Commit message: Actualizar archivos de descripción del robot para unificar rutas y corregir nombres de joints en los archivos URDF y XACRO. Arreglo de movimiento y limites del robot y nombres articualres.

File: src/robot_description/urdf/base_link_v_respaldo.xacro (robot description, xacro)
@@ -1,7 +1,7 @@
 <?xml version="1.0" ?>
 <robot name="base_link_v_respaldo" xmlns:xacro="http://www.ros.org/wiki/xacro">
-<xacro:include filename="$(find base_link_v_respaldo_description)/urdf/materials.xacro" />
-<xacro:include filename="$(find base_link_v_respaldo_description)/urdf/base_link_v_respaldo.trans" />
-<xacro:include filename="$(find base_link_v_respaldo_description)/urdf/base_link_v_respaldo.gazebo" />
+<xacro:include filename="$(find robot_description)/urdf/materials.xacro" />
+<xacro:include filename="$(find robot_description)/urdf/base_link_v_respaldo.trans" />
+<xacro:include filename="$(find robot_description)/urdf/base_link_v_respaldo.gazebo" />
 <link name="base_link">
   <inertial>
@@ -13,5 +13,5 @@
     <origin xyz="0 0 0" rpy="0 0 0"/>
     <geometry>
-      <mesh filename="package://base_link_v_respaldo_description/meshes/base_link.stl" scale="0.001 0.001 0.001"/>
+      <mesh filename="package://robot_description/meshes/base_link.stl" scale="0.001 0.001 0.001"/>
     </geometry>
     <material name="silver"/>
@@ -20,5 +20,5 @@
     <origin xyz="0 0 0" rpy="0 0 0"/>
     <geometry>
-      <mesh filename="package://base_link_v_respaldo_description/meshes/base_link.stl" scale="0.001 0.001 0.001"/>
+      <mesh filename="package://robot_description/meshes/base_link.stl" scale="0.001 0.001 0.001"/>
     </geometry>
   </collision>
@@ -33,5 +33,5 @@
     <origin xyz="-2.0 0.04 -0.72" rpy="0 0 0"/>
     <geometry>
-      <mesh filename="package://base_link_v_respaldo_description/meshes/carro_x_der_1_1.stl" scale="0.001 0.001 0.001"/>
+      <mesh filename="package://robot_description/meshes/carro_x_der_1_1.stl" scale="0.001 0.001 0.001"/>
     </geometry>
     <material name="silver"/>
@@ -40,5 +40,5 @@
     <origin xyz="-2.0 0.04 -0.72" rpy="0 0 0"/>
     <geometry>
-      <mesh filename="package://base_link_v_respaldo_description/meshes/carro_x_der_1_1.stl" scale="0.001 0.001 0.001"/>
+      <mesh filename="package://robot_description/meshes/carro_x_der_1_1.stl" scale="0.001 0.001 0.001"/>
     </geometry>
   </collision>
@@ -53,5 +53,5 @@
     <origin xyz="0.0 0.04 -0.72" rpy="0 0 0"/>
     <geometry>
-      <mesh filename="package://base_link_v_respaldo_description/meshes/carro_x_izq_1_1.stl" scale="0.001 0.001 0.001"/>
+      <mesh filename="package://robot_description/meshes/carro_x_izq_1_1.stl" scale="0.001 0.001 0.001"/>
     </geometry>
     <material name="silver"/>
@@ -60,5 +60,5 @@
     <origin xyz="0.0 0.04 -0.72" rpy="0 0 0"/>
     <geometry>
-      <mesh filename="package://base_link_v_respaldo_description/meshes/carro_x_izq_1_1.stl" scale="0.001 0.001 0.001"/>
+      <mesh filename="package://robot_description/meshes/carro_x_izq_1_1.stl" scale="0.001 0.001 0.001"/>
     </geometry>
   </collision>
@@ -73,5 +73,5 @@
     <origin xyz="-0.025 0.04 -0.64" rpy="0 0 0"/>
     <geometry>
-      <mesh filename="package://base_link_v_respaldo_description/meshes/base_y_izq_1_1.stl" scale="0.001 0.001 0.001"/>
+      <mesh filename="package://robot_description/meshes/base_y_izq_1_1.stl" scale="0.001 0.001 0.001"/>
     </geometry>
     <material name="silver"/>
@@ -80,5 +80,5 @@
     <origin xyz="-0.025 0.04 -0.64" rpy="0 0 0"/>
     <geometry>
-      <mesh filename="package://base_link_v_respaldo_description/meshes/base_y_izq_1_1.stl" scale="0.001 0.001 0.001"/>
+      <mesh filename="package://robot_description/meshes/base_y_izq_1_1.stl" scale="0.001 0.001 0.001"/>
     </geometry>
   </collision>
@@ -93,5 +93,5 @@
     <origin xyz="-1.975 0.04 -0.64" rpy="0 0 0"/>
     <geometry>
-      <mesh filename="package://base_link_v_respaldo_description/meshes/base_y_der_1_1.stl" scale="0.001 0.001 0.001"/>
+      <mesh filename="package://robot_description/meshes/base_y_der_1_1.stl" scale="0.001 0.001 0.001"/>
     </geometry>
     <material name="silver"/>
@@ -100,25 +100,5 @@
     <origin xyz="-1.975 0.04 -0.64" rpy="0 0 0"/>
     <geometry>
-      <mesh filename="package://base_link_v_respaldo_description/meshes/base_y_der_1_1.stl" scale="0.001 0.001 0.001"/>
-    </geometry>
-  </collision>
-</link>
-<link name="eje_carro_y_1_1">
-  <inertial>
-    <origin xyz="-0.9750000407869023 -0.01250028156917038 -0.040000044678056845" rpy="0 0 0"/>
-    <mass value="30.614999999998826"/>
-    <inertia ixx="0.017923" iyy="9.717456" izz="9.702723" ixy="0.0" iyz="0.0" ixz="0.0"/>
-  </inertial>
-  <visual>
-    <origin xyz="-1.897721 -0.733742 -1.456073" rpy="0 0 0"/>
-    <geometry>
-      <mesh filename="package://base_link_v_respaldo_description/meshes/eje_carro_y_1_1.stl" scale="0.001 0.001 0.001"/>
-    </geometry>
-    <material name="silver"/>
-  </visual>
-  <collision>
-    <origin xyz="-1.897721 -0.733742 -1.456073" rpy="0 0 0"/>
-    <geometry>
-      <mesh filename="package://base_link_v_respaldo_description/meshes/eje_carro_y_1_1.stl" scale="0.001 0.001 0.001"/>
+      <mesh filename="package://robot_description/meshes/base_y_der_1_1.stl" scale="0.001 0.001 0.001"/>
     </geometry>
   </collision>
@@ -133,5 +113,5 @@
     <origin xyz="0.052279 -0.733742 -1.456073" rpy="0 0 0"/>
     <geometry>
-      <mesh filename="package://base_link_v_respaldo_description/meshes/eje_carro_y_1_1.stl" scale="0.001 0.001 0.001"/>
+      <mesh filename="package://robot_description/meshes/eje_carro_y_1_1.stl" scale="0.001 0.001 0.001"/>
     </geometry>
     <material name="silver"/>
@@ -140,5 +120,5 @@
     <origin xyz="0.052279 -0.733742 -1.456073" rpy="0 0 0"/>
     <geometry>
-      <mesh filename="package://base_link_v_respaldo_description/meshes/eje_carro_y_1_1.stl" scale="0.001 0.001 0.001"/>
+      <mesh filename="package://robot_description/meshes/eje_carro_y_1_1.stl" scale="0.001 0.001 0.001"/>
     </geometry>
   </collision>
@@ -153,5 +133,5 @@
     <origin xyz="0.052279 -0.708742 -1.456073" rpy="0 0 0"/>
     <geometry>
-      <mesh filename="package://base_link_v_respaldo_description/meshes/carro_y_1_1.stl" scale="0.001 0.001 0.001"/>
+      <mesh filename="package://robot_description/meshes/carro_y_1_1.stl" scale="0.001 0.001 0.001"/>
     </geometry>
     <material name="silver"/>
@@ -160,5 +140,5 @@
     <origin xyz="0.052279 -0.708742 -1.456073" rpy="0 0 0"/>
     <geometry>
-      <mesh filename="package://base_link_v_respaldo_description/meshes/carro_y_1_1.stl" scale="0.001 0.001 0.001"/>
+      <mesh filename="package://robot_description/meshes/carro_y_1_1.stl" scale="0.001 0.001 0.001"/>
     </geometry>
   </collision>
@@ -173,5 +153,5 @@
     <origin xyz="-0.509116 -0.683742 -1.456073" rpy="0 0 0"/>
     <geometry>
-      <mesh filename="package://base_link_v_respaldo_description/meshes/carro_z_1_1.stl" scale="0.001 0.001 0.001"/>
+      <mesh filename="package://robot_description/meshes/carro_z_1_1.stl" scale="0.001 0.001 0.001"/>
     </geometry>
     <material name="silver"/>
@@ -180,5 +160,5 @@
     <origin xyz="-0.509116 -0.683742 -1.456073" rpy="0 0 0"/>
     <geometry>
-      <mesh filename="package://base_link_v_respaldo_description/meshes/carro_z_1_1.stl" scale="0.001 0.001 0.001"/>
+      <mesh filename="package://robot_description/meshes/carro_z_1_1.stl" scale="0.001 0.001 0.001"/>
     </geometry>
   </collision>
@@ -193,5 +173,5 @@
     <origin xyz="-0.509116 -0.658742 -0.591602" rpy="0 0 0"/>
     <geometry>
-      <mesh filename="package://base_link_v_respaldo_description/meshes/soporte_camara_1_1.stl" scale="0.001 0.001 0.001"/>
+      <mesh filename="package://robot_description/meshes/soporte_camara_1_1.stl" scale="0.001 0.001 0.001"/>
     </geometry>
     <material name="silver"/>
@@ -200,5 +180,5 @@
     <origin xyz="-0.509116 -0.658742 -0.591602" rpy="0 0 0"/>
     <geometry>
-      <mesh filename="package://base_link_v_respaldo_description/meshes/soporte_camara_1_1.stl" scale="0.001 0.001 0.001"/>
+      <mesh filename="package://robot_description/meshes/soporte_camara_1_1.stl" scale="0.001 0.001 0.001"/>
     </geometry>
   </collision>
@@ -213,5 +193,5 @@
     <origin xyz="-0.509116 -0.658742 -0.591602" rpy="0 0 0"/>
     <geometry>
-      <mesh filename="package://base_link_v_respaldo_description/meshes/base_muneca_1_1.stl" scale="0.001 0.001 0.001"/>
+      <mesh filename="package://robot_description/meshes/base_muneca_1_1.stl" scale="0.001 0.001 0.001"/>
     </geometry>
     <material name="silver"/>
@@ -220,5 +200,5 @@
     <origin xyz="-0.509116 -0.658742 -0.591602" rpy="0 0 0"/>
     <geometry>
-      <mesh filename="package://base_link_v_respaldo_description/meshes/base_muneca_1_1.stl" scale="0.001 0.001 0.001"/>
+      <mesh filename="package://robot_description/meshes/base_muneca_1_1.stl" scale="0.001 0.001 0.001"/>
     </geometry>
   </collision>
@@ -233,5 +213,5 @@
     <origin xyz="-0.652234 -0.367376 -0.402215" rpy="0 0 0"/>
     <geometry>
-      <mesh filename="package://base_link_v_respaldo_description/meshes/eje_muneca_izq_1.stl" scale="0.001 0.001 0.001"/>
+      <mesh filename="package://robot_description/meshes/eje_muneca_izq_1.stl" scale="0.001 0.001 0.001"/>
     </geometry>
     <material name="silver"/>
@@ -240,5 +220,5 @@
     <origin xyz="-0.652234 -0.367376 -0.402215" rpy="0 0 0"/>
     <geometry>
-      <mesh filename="package://base_link_v_respaldo_description/meshes/eje_muneca_izq_1.stl" scale="0.001 0.001 0.001"/>
+      <mesh filename="package://robot_description/meshes/eje_muneca_izq_1.stl" scale="0.001 0.001 0.001"/>
     </geometry>
   </collision>
@@ -253,5 +233,5 @@
     <origin xyz="-0.732234 -0.367376 -0.362215" rpy="0 0 0"/>
     <geometry>
-      <mesh filename="package://base_link_v_respaldo_description/meshes/eje_muneca_der_1_1.stl" scale="0.001 0.001 0.001"/>
+      <mesh filename="package://robot_description/meshes/eje_muneca_der_1_1.stl" scale="0.001 0.001 0.001"/>
     </geometry>
     <material name="silver"/>
@@ -260,5 +240,5 @@
     <origin xyz="-0.732234 -0.367376 -0.362215" rpy="0 0 0"/>
     <geometry>
-      <mesh filename="package://base_link_v_respaldo_description/meshes/eje_muneca_der_1_1.stl" scale="0.001 0.001 0.001"/>
+      <mesh filename="package://robot_description/meshes/eje_muneca_der_1_1.stl" scale="0.001 0.001 0.001"/>
     </geometry>
   </collision>
@@ -273,5 +253,5 @@
     <origin xyz="-0.744269 -0.900107 -1.080989" rpy="0 0 0"/>
     <geometry>
-      <mesh filename="package://base_link_v_respaldo_description/meshes/paleta_muneca_der_1.stl" scale="0.001 0.001 0.001"/>
+      <mesh filename="package://robot_description/meshes/paleta_muneca_der_1.stl" scale="0.001 0.001 0.001"/>
     </geometry>
     <material name="silver"/>
@@ -280,5 +260,5 @@
     <origin xyz="-0.744269 -0.900107 -1.080989" rpy="0 0 0"/>
     <geometry>
-      <mesh filename="package://base_link_v_respaldo_description/meshes/paleta_muneca_der_1.stl" scale="0.001 0.001 0.001"/>
+      <mesh filename="package://robot_description/meshes/paleta_muneca_der_1.stl" scale="0.001 0.001 0.001"/>
     </geometry>
   </collision>
@@ -293,5 +273,5 @@
     <origin xyz="-0.207876 -0.392484 -1.069671" rpy="0 0 0"/>
     <geometry>
-      <mesh filename="package://base_link_v_respaldo_description/meshes/paleta_muneca_izq_1_1.stl" scale="0.001 0.001 0.001"/>
+      <mesh filename="package://robot_description/meshes/paleta_muneca_izq_1_1.stl" scale="0.001 0.001 0.001"/>
     </geometry>
     <material name="silver"/>
@@ -300,5 +280,5 @@
     <origin xyz="-0.207876 -0.392484 -1.069671" rpy="0 0 0"/>
     <geometry>
-      <mesh filename="package://base_link_v_respaldo_description/meshes/paleta_muneca_izq_1_1.stl" scale="0.001 0.001 0.001"/>
+      <mesh filename="package://robot_description/meshes/paleta_muneca_izq_1_1.stl" scale="0.001 0.001 0.001"/>
     </geometry>
   </collision>
@@ -313,5 +293,5 @@
     <origin xyz="0.0 0.04 -0.64" rpy="0 0 0"/>
     <geometry>
-      <mesh filename="package://base_link_v_respaldo_description/meshes/base_eje_x_izq_1_1.stl" scale="0.001 0.001 0.001"/>
+      <mesh filename="package://robot_description/meshes/base_eje_x_izq_1_1.stl" scale="0.001 0.001 0.001"/>
     </geometry>
     <material name="silver"/>
@@ -320,5 +300,5 @@
     <origin xyz="0.0 0.04 -0.64" rpy="0 0 0"/>
     <geometry>
-      <mesh filename="package://base_link_v_respaldo_description/meshes/base_eje_x_izq_1_1.stl" scale="0.001 0.001 0.001"/>
+      <mesh filename="package://robot_description/meshes/base_eje_x_izq_1_1.stl" scale="0.001 0.001 0.001"/>
     </geometry>
   </collision>
@@ -333,5 +313,5 @@
     <origin xyz="-2.04 0.04 -0.64" rpy="0 0 0"/>
     <geometry>
-      <mesh filename="package://base_link_v_respaldo_description/meshes/base_eje_x_der_1_1.stl" scale="0.001 0.001 0.001"/>
+      <mesh filename="package://robot_description/meshes/base_eje_x_der_1_1.stl" scale="0.001 0.001 0.001"/>
     </geometry>
     <material name="silver"/>
@@ -340,16 +320,16 @@
     <origin xyz="-2.04 0.04 -0.64" rpy="0 0 0"/>
     <geometry>
-      <mesh filename="package://base_link_v_respaldo_description/meshes/base_eje_x_der_1_1.stl" scale="0.001 0.001 0.001"/>
-    </geometry>
-  </collision>
-</link>
-<joint name="Corredera 3" type="prismatic">
+      <mesh filename="package://robot_description/meshes/base_eje_x_der_1_1.stl" scale="0.001 0.001 0.001"/>
+    </geometry>
+  </collision>
+</link>
+<joint name="Eje x" type="prismatic">
   <origin xyz="-0.04 0.0 0.08" rpy="0 0 0"/>
   <parent link="base_eje_x_der_1_1"/>
   <child link="carro_x_der_1_1"/>
   <axis xyz="-0.0 -1.0 0.0"/>
-  <limit upper="-0.2" lower="-1.75" effort="100" velocity="100"/>
-</joint>
-<joint name="Corredera 4" type="prismatic">
+  <limit upper="+0.2" lower="-0.40" effort="100" velocity="100"/>
+</joint>
+<joint name="Eje x copia" type="prismatic">
   <origin xyz="0.0 0.0 0.08" rpy="0 0 0"/>
   <parent link="base_eje_x_izq_1_1"/>
@@ -357,33 +337,34 @@
   <axis xyz="0.0 1.0 -0.0"/>
   <limit upper="0.75" lower="0.2" effort="100" velocity="100"/>
-</joint>
-<joint name="R�gida 5" type="fixed">
+  <mimic joint="Eje x" multiplier="-1.0" offset="0.0"/>
+</joint>
+<joint name="Rigida 5" type="fixed">
   <origin xyz="0.025 0.0 -0.08" rpy="0 0 0"/>
   <parent link="carro_x_izq_1_1"/>
   <child link="base_y_izq_1_1"/>
 </joint>
-<joint name="R�gida 6" type="fixed">
+<joint name="Rigida 6" type="fixed">
   <origin xyz="-0.025 0.0 -0.08" rpy="0 0 0"/>
   <parent link="carro_x_der_1_1"/>
   <child link="base_y_der_1_1"/>
 </joint>
-<joint name="R�gida 7" type="fixed">
+<joint name="Rigida 7" type="fixed">
   <origin xyz="-2.027279 0.773742 0.816073" rpy="0 0 0"/>
   <parent link="base_y_der_1_1"/>
   <child link="eje_carro_y_1_1"/>
 </joint>
-<joint name="R�gida 8" type="fixed">
+<joint name="Rigida 8" type="fixed">
   <origin xyz="-0.077279 0.773742 0.816073" rpy="0 0 0"/>
   <parent link="base_y_izq_1_1"/>
   <child link="eje_carro_y_1_1"/>
 </joint>
-<joint name="Corredera 9" type="prismatic">
+<joint name="Eje y" type="prismatic">
   <origin xyz="0.0 -0.025 0.0" rpy="0 0 0"/>
   <parent link="eje_carro_y_1_1"/>
   <child link="carro_y_1_1"/>
   <axis xyz="1.0 0.0 0.0"/>
-  <limit upper="1.7" lower="0.2" effort="100" velocity="100"/>
-</joint>
-<joint name="Corredera 10" type="prismatic">
+  <limit upper="0.71" lower="-0.75" effort="100" velocity="100"/>
+</joint>
+<joint name="Eje z" type="prismatic">
   <origin xyz="0.561395 -0.025 0.0" rpy="0 0 0"/>
   <parent link="carro_y_1_1"/>
@@ -392,20 +373,20 @@
   <limit upper="-0.05" lower="-1.0" effort="100" velocity="100"/>
 </joint>
-<joint name="R�gida 11" type="fixed">
+<joint name="Rigida 11" type="fixed">
   <origin xyz="0.0 -0.025 -0.864471" rpy="0 0 0"/>
   <parent link="carro_z_1_1"/>
   <child link="soporte_camara_1_1"/>
 </joint>
-<joint name="R�gida 12" type="fixed">
+<joint name="Rigida 12" type="fixed">
   <origin xyz="0.0 -0.025 -0.864471" rpy="0 0 0"/>
   <parent link="carro_z_1_1"/>
   <child link="base_muneca_1_1"/>
 </joint>
-<joint name="Corredera 13" type="prismatic">
+<joint name="muneca" type="prismatic">
   <origin xyz="0.143118 -0.291366 -0.189387" rpy="0 0 0"/>
   <parent link="base_muneca_1_1"/>
   <child link="eje_muneca_izq_1"/>
   <axis xyz="-1.0 0.0 -0.0"/>
-  <limit upper="-0.08" lower="-0.14" effort="100" velocity="100"/>
+  <limit upper="+0.08" lower="-0.05" effort="100" velocity="100"/>
 </joint>
 <joint name="Corredera 14" type="prismatic">
@@ -414,22 +395,23 @@
   <child link="eje_muneca_der_1_1"/>
   <axis xyz="1.0 -0.0 0.0"/>
-  <limit upper="-0.08" lower="-0.14" effort="100" velocity="100"/>
-</joint>
-<joint name="R�gida 15" type="fixed">
+  <limit upper="+0.08" lower="-0.05" effort="100" velocity="100"/>
+    <mimic joint="muneca" multiplier="+1.0" offset="0.0"/>
+</joint>
+<joint name="Rigida 15" type="fixed">
   <origin xyz="0.012035 0.532731 0.718774" rpy="0 0 0"/>
   <parent link="eje_muneca_der_1_1"/>
   <child link="paleta_muneca_der_1"/>
 </joint>
-<joint name="R�gida 16" type="fixed">
+<joint name="Rigida 16" type="fixed">
   <origin xyz="-0.444358 0.025108 0.667456" rpy="0 0 0"/>
   <parent link="eje_muneca_izq_1"/>
   <child link="paleta_muneca_izq_1_1"/>
 </joint>
-<joint name="R�gida 17" type="fixed">
+<joint name="Rigida 17" type="fixed">
   <origin xyz="0.0 -0.04 0.64" rpy="0 0 0"/>
   <parent link="base_link"/>
   <child link="base_eje_x_izq_1_1"/>
 </joint>
-<joint name="R�gida 18" type="fixed">
+<joint name="Rigida 18" type="fixed">
   <origin xyz="2.04 -0.04 0.64" rpy="0 0 0"/>
   <parent link="base_link"/>
