Commit message: Añade documentación sobre la importación del robot en NVIDIA Isaac Sim y actualiza el archivo URDF para incluir el modelo completo.

File: src/robot_description/urdf/robot_description_isaac.urdf (robot description, URDF)
Before this commit: robot robot_description, 4 links, 3 joints
Links:
- added link Externo1_v1_1, mass 3.103290090272312; collision mesh filename=../meshes/Externo1_v1_1.stl scale=0.001 0.001 0.001; visual mesh filename=../meshes/Externo1_v1_1.stl scale=0.001 0.001 0.001
- added link Externo3_v1_1_1, mass 0.07977197198617901; collision mesh filename=../meshes/Externo3_v1_1_1.stl scale=0.001 0.001 0.001; visual mesh filename=../meshes/Externo3_v1_1_1.stl scale=0.001 0.001 0.001
- added link Pala_DER_1, mass 1.1995109762545986; collision mesh filename=../meshes/Pala_DER_1.stl scale=0.001 0.001 0.001; visual mesh filename=../meshes/Pala_DER_1.stl scale=0.001 0.001 0.001
- added link Pala_IZQ_1, mass 1.1995109762545986; collision mesh filename=../meshes/Pala_IZQ_1.stl scale=0.001 0.001 0.001; visual mesh filename=../meshes/Pala_IZQ_1.stl scale=0.001 0.001 0.001
- added link Paleta_1_1, mass 0.3818616414823265; collision mesh filename=../meshes/Paleta_1_1.stl scale=0.001 0.001 0.001; visual mesh filename=../meshes/Paleta_1_1.stl scale=0.001 0.001 0.001
- added link Paleta_2_1, mass 0.3818616414823265; collision mesh filename=../meshes/Paleta_2_1.stl scale=0.001 0.001 0.001; visual mesh filename=../meshes/Paleta_2_1.stl scale=0.001 0.001 0.001
- added link Servo_horn_v2_v1_1, mass 0.005099610361289279; collision mesh filename=../meshes/Servo_horn_v2_v1_1.stl scale=0.001 0.001 0.001; visual mesh filename=../meshes/Servo_horn_v2_v1_1.stl scale=0.001 0.001 0.001
- added link cabezal_1, mass 5.246895030843086; collision mesh filename=../meshes/cabezal_1.stl scale=0.001 0.001 0.001; visual mesh filename=../meshes/cabezal_1.stl scale=0.001 0.001 0.001
- added link cabezal_2_0_v1_1_1, mass 5.768314857333685; collision mesh filename=../meshes/cabezal_2.0_v1_1_1.stl scale=0.001 0.001 0.001; visual mesh filename=../meshes/cabezal_2.0_v1_1_1.stl scale=0.001 0.001 0.001
- added link mg996R_v2_v1_1_1, mass 0.24706045427040543; collision mesh filename=../meshes/mg996R_v2_v1_1_1.stl scale=0.001 0.001 0.001; visual mesh filename=../meshes/mg996R_v2_v1_1_1.stl scale=0.001 0.001 0.001
- link y_link_1: mass 0.29493075116533896 -> 0.5775307511653394
Joints:
- added joint Grid_DER: type prismatic, parent Externo3_v1_1_1, child Paleta_2_1, origin xyz=0.025022 -0.00489 0.0 rpy=0 0 0, axis -0.99999 -0.004384 0.0, limit lower=0.0 upper=0.04 effort=100 velocity=100
- added joint Grid_IZQ: type prismatic, parent Externo3_v1_1_1, child Paleta_1_1, origin xyz=-0.024978 -0.00511 0.0 rpy=0 0 0, axis -0.99999 -0.004384 0.0, limit lower=-0.040 upper=0.0 effort=100 velocity=100, mimic joint=Grid_DER multiplier=-1 offset=0
- added joint R_joint: type continuous, parent cabezal_1, child Externo1_v1_1, origin xyz=0.0 -0.05 0.0145 rpy=0 0 0, axis -0.0 -0.0 -1.0
- added joint Rig_1: type fixed, parent z_link_1, child cabezal_1, origin xyz=0.0 -0.04 -1.025 rpy=0 0 0
- added joint Rig_2: type fixed, parent Externo1_v1_1, child cabezal_2_0_v1_1_1, origin xyz=0.0 0.0 -0.0495 rpy=0 0 0
- added joint Rig_3: type fixed, parent cabezal_2_0_v1_1_1, child mg996R_v2_v1_1_1, origin xyz=0.00491 0.020522 -0.1155 rpy=0 0 0
- added joint Rig_4: type fixed, parent mg996R_v2_v1_1_1, child Servo_horn_v2_v1_1, origin xyz=-0.004949 -0.011522 0.0345 rpy=0 0 0
- added joint Rig_5: type fixed, parent Servo_horn_v2_v1_1, child Externo3_v1_1_1, origin xyz=1.9e-05 -0.0045 0.0 rpy=0 0 0
- added joint Rig_6: type fixed, parent Paleta_1_1, child Pala_IZQ_1, origin xyz=-0.213998 -0.000938 0.0 rpy=0 0 0
- added joint Rig_7: type fixed, parent Paleta_2_1, child Pala_DER_1, origin xyz=0.213998 0.000938 0.0 rpy=0 0 0
- joint x_joint: limit lower=0.02 upper=0.94 effort=100 velocity=100 -> lower=0.02 upper=0.94 effort=10000 velocity=1000
- joint y_joint: limit lower=0.065 upper=0.838 effort=100 velocity=100 -> lower=0.065 upper=0.838 effort=10000 velocity=1000
- joint z_joint: axis 0.0 -0.0 1.0 -> -0.0 -0.0 -1.0; limit lower=0.0 upper=0.93 effort=100 velocity=100 -> lower=-0.93 upper=0 effort=10000 velocity=1000; origin xyz=0.08 -0.0025 0.09 rpy=0 0 0 -> xyz=0.08 -0.0075 0.09 rpy=0 0 0
