Commit message: actualizacion de limite de ejes y limpiesza de archivos antiguos

File: src/robot_description/urdf/robot.xacro (robot description, xacro)
@@ -306,5 +306,5 @@
 </joint>
 <joint name="Rig_1" type="fixed">
-  <origin xyz="0.0 -0.04 -1.025" rpy="0 0 0"/>
+  <origin xyz="-0.04 -0.04 -1.025" rpy="0 0 0"/>
   <parent link="z_link_1"/>
   <child link="cabezal_1"/>

File: src/robot_description/urdf/robot_isaac.urdf (robot description, URDF)
Before this commit: robot robot, 14 links, 13 joints
Joints:
- joint Rig_1: origin xyz=0.0 -0.04 -1.025 rpy=0 0 0 -> xyz=-0.04 -0.04 -1.025 rpy=0 0 0

Commit message: Add USD files for robot_isaac configuration and physics
- Created robot_isaac_base.usd to define the base configuration of the robot.
- Added robot_isaac_physics.usd to specify the physics properties of the robot.
- Introduced robot_isaac_sensor.usd for sensor configurations.
- Updated robot_isaac.usd to include references to the new configuration files.

File: src/robot_description/urdf/robot.xacro (robot description, xacro)
@@ -1,7 +1,15 @@
 <?xml version="1.0" ?>
 <robot name="robot" xmlns:xacro="http://www.ros.org/wiki/xacro">
+<xacro:arg name="include_transmissions" default="true"/>
+<xacro:arg name="include_gazebo" default="true"/>
+<xacro:arg name="mesh_directory" default="file://$(find robot_description)/meshes"/>
+<xacro:property name="mesh_directory" value="$(arg mesh_directory)"/>
 <xacro:include filename="$(find robot_description)/urdf/materials.xacro" />
-<xacro:include filename="$(find robot_description)/urdf/robot.trans" />
-<xacro:include filename="$(find robot_description)/urdf/robot.gazebo" />
+<xacro:if value="$(arg include_transmissions)">
+  <xacro:include filename="$(find robot_description)/urdf/robot.trans" />
+</xacro:if>
+<xacro:if value="$(arg include_gazebo)">
+  <xacro:include filename="$(find robot_description)/urdf/robot.gazebo" />
+</xacro:if>
 <link name="base_link">
   <inertial>
@@ -13,5 +21,5 @@
     <origin xyz="0 0 0" rpy="0 0 0"/>
     <geometry>
-      <mesh filename="file://$(find robot_description)/meshes/base_link.stl" scale="0.001 0.001 0.001"/>
+      <mesh filename="${mesh_directory}/base_link.stl" scale="0.001 0.001 0.001"/>
     </geometry>
     <material name="silver"/>
@@ -20,5 +28,5 @@
     <origin xyz="0 0 0" rpy="0 0 0"/>
     <geometry>
-      <mesh filename="file://$(find robot_description)/meshes/base_link.stl" scale="0.001 0.001 0.001"/>
+      <mesh filename="${mesh_directory}/base_link.stl" scale="0.001 0.001 0.001"/>
     </geometry>
   </collision>
@@ -33,5 +41,5 @@
     <origin xyz="-0.0285 -0.0 -0.603" rpy="0 0 0"/>
     <geometry>
-      <mesh filename="file://$(find robot_description)/meshes/x_link_1.stl" scale="0.001 0.001 0.001"/>
+      <mesh filename="${mesh_directory}/x_link_1.stl" scale="0.001 0.001 0.001"/>
     </geometry>
     <material name="silver"/>
@@ -40,5 +48,5 @@
     <origin xyz="-0.0285 -0.0 -0.603" rpy="0 0 0"/>
     <geometry>
-      <mesh filename="file://$(find robot_description)/meshes/x_link_1.stl" scale="0.001 0.001 0.001"/>
+      <mesh filename="${mesh_directory}/x_link_1.stl" scale="0.001 0.001 0.001"/>
     </geometry>
   </collision>
@@ -53,5 +61,5 @@
     <origin xyz="0.034 0.12 -1.081" rpy="0 0 0"/>
     <geometry>
-      <mesh filename="file://$(find robot_description)/meshes/y_link_1.stl" scale="0.001 0.001 0.001"/>
+      <mesh filename="${mesh_directory}/y_link_1.stl" scale="0.001 0.001 0.001"/>
     </geometry>
     <material name="silver"/>
@@ -60,5 +68,5 @@
     <origin xyz="0.034 0.12 -1.081" rpy="0 0 0"/>
     <geometry>
-      <mesh filename="file://$(find robot_description)/meshes/y_link_1.stl" scale="0.001 0.001 0.001"/>
+      <mesh filename="${mesh_directory}/y_link_1.stl" scale="0.001 0.001 0.001"/>
     </geometry>
   </collision>
@@ -73,5 +81,5 @@
     <origin xyz="-0.046 0.1275 -1.171" rpy="0 0 0"/>
     <geometry>
-      <mesh filename="file://$(find robot_description)/meshes/z_link_1.stl" scale="0.001 0.001 0.001"/>
+      <mesh filename="${mesh_directory}/z_link_1.stl" scale="0.001 0.001 0.001"/>
     </geometry>
     <material name="silver"/>
@@ -80,5 +88,5 @@
     <origin xyz="-0.046 0.1275 -1.171" rpy="0 0 0"/>
     <geometry>
-      <mesh filename="file://$(find robot_description)/meshes/z_link_1.stl" scale="0.001 0.001 0.001"/>
+      <mesh filename="${mesh_directory}/z_link_1.stl" scale="0.001 0.001 0.001"/>
     </geometry>
   </collision>
@@ -93,5 +101,5 @@
     <origin xyz="-0.046 0.1675 -0.146" rpy="0 0 0"/>
     <geometry>
-      <mesh filename="file://$(find robot_description)/meshes/cabezal_1.stl" scale="0.001 0.001 0.001"/>
+      <mesh filename="${mesh_directory}/cabezal_1.stl" scale="0.001 0.001 0.001"/>
     </geometry>
     <material name="silver"/>
@@ -100,5 +108,5 @@
     <origin xyz="-0.046 0.1675 -0.146" rpy="0 0 0"/>
     <geometry>
-      <mesh filename="file://$(find robot_description)/meshes/cabezal_1.stl" scale="0.001 0.001 0.001"/>
+      <mesh filename="${mesh_directory}/cabezal_1.stl" scale="0.001 0.001 0.001"/>
     </geometry>
   </collision>
@@ -113,5 +121,5 @@
     <origin xyz="-0.046 0.2175 -0.1605" rpy="0 0 0"/>
     <geometry>
-      <mesh filename="file://$(find robot_description)/meshes/Externo1_v1_1.stl" scale="0.001 0.001 0.001"/>
+      <mesh filename="${mesh_directory}/Externo1_v1_1.stl" scale="0.001 0.001 0.001"/>
     </geometry>
     <material name="silver"/>
@@ -120,9 +128,9 @@
     <origin xyz="-0.046 0.2175 -0.1605" rpy="0 0 0"/>
     <geometry>
-      <mesh filename="file://$(find robot_description)/meshes/Externo1_v1_1.stl" scale="0.001 0.001 0.001"/>
-    </geometry>
-  </collision>
-</link>
-<link name="cabezal_2.0_v1_1_1">
+      <mesh filename="${mesh_directory}/Externo1_v1_1.stl" scale="0.001 0.001 0.001"/>
+    </geometry>
+  </collision>
+</link>
+<link name="cabezal_2_0_v1_1_1">
   <inertial>
     <origin xyz="-1.9836844046515478e-05 0.00327884619901872 -0.05001506846643826" rpy="0 0 0"/>
@@ -133,5 +141,5 @@
     <origin xyz="-0.046 0.2175 -0.111" rpy="0 0 0"/>
     <geometry>
-      <mesh filename="file://$(find robot_description)/meshes/cabezal_2.0_v1_1_1.stl" scale="0.001 0.001 0.001"/>
+      <mesh filename="${mesh_directory}/cabezal_2_0_v1_1_1.stl" scale="0.001 0.001 0.001"/>
     </geometry>
     <material name="silver"/>
@@ -140,5 +148,5 @@
     <origin xyz="-0.046 0.2175 -0.111" rpy="0 0 0"/>
     <geometry>
-      <mesh filename="file://$(find robot_description)/meshes/cabezal_2.0_v1_1_1.stl" scale="0.001 0.001 0.001"/>
+      <mesh filename="${mesh_directory}/cabezal_2_0_v1_1_1.stl" scale="0.001 0.001 0.001"/>
     </geometry>
   </collision>
@@ -153,5 +161,5 @@
     <origin xyz="-0.05091 0.196978 0.0045" rpy="0 0 0"/>
     <geometry>
-      <mesh filename="file://$(find robot_description)/meshes/mg996R_v2_v1_1_1.stl" scale="0.001 0.001 0.001"/>
+      <mesh filename="${mesh_directory}/mg996R_v2_v1_1_1.stl" scale="0.001 0.001 0.001"/>
     </geometry>
     <material name="silver"/>
@@ -160,5 +168,5 @@
     <origin xyz="-0.05091 0.196978 0.0045" rpy="0 0 0"/>
     <geometry>
-      <mesh filename="file://$(find robot_description)/meshes/mg996R_v2_v1_1_1.stl" scale="0.001 0.001 0.001"/>
+      <mesh filename="${mesh_directory}/mg996R_v2_v1_1_1.stl" scale="0.001 0.001 0.001"/>
     </geometry>
   </collision>
@@ -168,10 +176,10 @@
     <origin xyz="1.3515116238912994e-05 -0.0031874939270762903 -1.5161483180037294e-15" rpy="0 0 0"/>
     <mass value="0.005099610361289279"/>
-    <inertia ixx="0.0" iyy="0.0" izz="0.0" ixy="-0.0" iyz="-0.0" ixz="0.0"/>
+    <inertia ixx="1.253100175e-07" iyy="2.404369626e-07" izz="1.253077337e-07" ixy="-5.047754088e-10" iyz="-7.092025118e-16" ixz="4.671074672e-16"/>
   </inertial>
   <visual>
     <origin xyz="-0.045961 0.2085 -0.03" rpy="0 0 0"/>
     <geometry>
-      <mesh filename="file://$(find robot_description)/meshes/Servo_horn_v2_v1_1.stl" scale="0.001 0.001 0.001"/>
+      <mesh filename="${mesh_directory}/Servo_horn_v2_v1_1.stl" scale="0.001 0.001 0.001"/>
     </geometry>
     <material name="silver"/>
@@ -180,5 +188,5 @@
     <origin xyz="-0.045961 0.2085 -0.03" rpy="0 0 0"/>
     <geometry>
-      <mesh filename="file://$(find robot_description)/meshes/Servo_horn_v2_v1_1.stl" scale="0.001 0.001 0.001"/>
+      <mesh filename="${mesh_directory}/Servo_horn_v2_v1_1.stl" scale="0.001 0.001 0.001"/>
     </geometry>
   </collision>
@@ -193,5 +201,5 @@
     <origin xyz="-0.04598 0.213 -0.03" rpy="0 0 0"/>
     <geometry>
-      <mesh filename="file://$(find robot_description)/meshes/Externo3_v1_1_1.stl" scale="0.001 0.001 0.001"/>
+      <mesh filename="${mesh_directory}/Externo3_v1_1_1.stl" scale="0.001 0.001 0.001"/>
     </geometry>
     <material name="silver"/>
@@ -200,5 +208,5 @@
     <origin xyz="-0.04598 0.213 -0.03" rpy="0 0 0"/>
     <geometry>
-      <mesh filename="file://$(find robot_description)/meshes/Externo3_v1_1_1.stl" scale="0.001 0.001 0.001"/>
+      <mesh filename="${mesh_directory}/Externo3_v1_1_1.stl" scale="0.001 0.001 0.001"/>
     </geometry>
   </collision>
@@ -213,5 +221,5 @@
     <origin xyz="-0.021002 0.21811 -0.03" rpy="0 0 0"/>
     <geometry>
-      <mesh filename="file://$(find robot_description)/meshes/Paleta_1_1.stl" scale="0.001 0.001 0.001"/>
+      <mesh filename="${mesh_directory}/Paleta_1_1.stl" scale="0.001 0.001 0.001"/>
     </geometry>
     <material name="silver"/>
@@ -220,5 +228,5 @@
     <origin xyz="-0.021002 0.21811 -0.03" rpy="0 0 0"/>
     <geometry>
-      <mesh filename="file://$(find robot_description)/meshes/Paleta_1_1.stl" scale="0.001 0.001 0.001"/>
+      <mesh filename="${mesh_directory}/Paleta_1_1.stl" scale="0.001 0.001 0.001"/>
     </geometry>
   </collision>
@@ -233,5 +241,5 @@
     <origin xyz="-0.071002 0.21789 -0.03" rpy="0 0 0"/>
     <geometry>
-      <mesh filename="file://$(find robot_description)/meshes/Paleta_2_1.stl" scale="0.001 0.001 0.001"/>
+      <mesh filename="${mesh_directory}/Paleta_2_1.stl" scale="0.001 0.001 0.001"/>
     </geometry>
     <material name="silver"/>
@@ -240,5 +248,5 @@
     <origin xyz="-0.071002 0.21789 -0.03" rpy="0 0 0"/>
     <geometry>
-      <mesh filename="file://$(find robot_description)/meshes/Paleta_2_1.stl" scale="0.001 0.001 0.001"/>
+      <mesh filename="${mesh_directory}/Paleta_2_1.stl" scale="0.001 0.001 0.001"/>
     </geometry>
   </collision>
@@ -253,5 +261,5 @@
     <origin xyz="0.192996 0.219048 -0.03" rpy="0 0 0"/>
     <geometry>
-      <mesh filename="file://$(find robot_description)/meshes/Pala_IZQ_1.stl" scale="0.001 0.001 0.001"/>
+      <mesh filename="${mesh_directory}/Pala_IZQ_1.stl" scale="0.001 0.001 0.001"/>
     </geometry>
     <material name="silver"/>
@@ -260,5 +268,5 @@
     <origin xyz="0.192996 0.219048 -0.03" rpy="0 0 0"/>
     <geometry>
-      <mesh filename="file://$(find robot_description)/meshes/Pala_IZQ_1.stl" scale="0.001 0.001 0.001"/>
+      <mesh filename="${mesh_directory}/Pala_IZQ_1.stl" scale="0.001 0.001 0.001"/>
     </geometry>
   </collision>
@@ -273,5 +281,5 @@
     <origin xyz="-0.285 0.216952 -0.03" rpy="0 0 0"/>
     <geometry>
-      <mesh filename="file://$(find robot_description)/meshes/Pala_DER_1.stl" scale="0.001 0.001 0.001"/>
+      <mesh filename="${mesh_directory}/Pala_DER_1.stl" scale="0.001 0.001 0.001"/>
     </geometry>
     <material name="silver"/>
@@ -280,5 +288,5 @@
     <origin xyz="-0.285 0.216952 -0.03" rpy="0 0 0"/>
     <geometry>
-      <mesh filename="file://$(find robot_description)/meshes/Pala_DER_1.stl" scale="0.001 0.001 0.001"/>
+      <mesh filename="${mesh_directory}/Pala_DER_1.stl" scale="0.001 0.001 0.001"/>
     </geometry>
   </collision>
@@ -319,9 +327,9 @@
   <origin xyz="0.0 0.0 -0.0495" rpy="0 0 0"/>
   <parent link="Externo1_v1_1"/>
-  <child link="cabezal_2.0_v1_1_1"/>
+  <child link="cabezal_2_0_v1_1_1"/>
 </joint>
 <joint name="Rig_3" type="fixed">
   <origin xyz="0.00491 0.020522 -0.1155" rpy="0 0 0"/>
-  <parent link="cabezal_2.0_v1_1_1"/>
+  <parent link="cabezal_2_0_v1_1_1"/>
   <child link="mg996R_v2_v1_1_1"/>
 </joint>

File: src/robot_description/urdf/robot_isaac.urdf (robot description, URDF)
Before this commit: robot robot, 14 links, 13 joints
Links:
- link cabezal_2_0_v1_1_1: geometry collision mesh filename=../meshes/cabezal_2_0_v1_1_1.stl scale=0.001 0.001 0.001; visual mesh filename=../meshes/cabezal_2_0_v1_1_1.stl scale=0.001 0.001 0.001

Commit message: Actaulizacion de robot.xacro con las masas, centros de masa y tensores de inercia

File: src/robot_description/urdf/robot.xacro (robot description, xacro)
@@ -6,7 +6,7 @@
 <link name="base_link">
   <inertial>
-    <origin xyz="0.45768622613563736 -0.4368264195359295 0.4295018217497949" rpy="0 0 0"/>
-    <mass value="145.80079322670187"/>
-    <inertia ixx="27.178522" iyy="35.333395" izz="48.362655" ixy="-0.011589" iyz="0.792709" ixz="-0.004434"/>
+    <origin xyz="0.45768622613563736 -0.4368264195359295 0.4295018217497948" rpy="0 0 0"/>
+    <mass value="50.148043530203196"/>
+    <inertia ixx="9.348027" iyy="12.152888" izz="16.634289" ixy="-0.003986" iyz="0.272652" ixz="-0.001525"/>
   </inertial>
   <visual>
@@ -26,7 +26,7 @@
 <link name="x_link_1">
   <inertial>
-    <origin xyz="0.42900000000000316 -0.07702054233668737 0.4385579778257891" rpy="0 0 0"/>
-    <mass value="33.63690371299227"/>
-    <inertia ixx="0.818102" iyy="5.092965" izz="4.355089" ixy="-1e-06" iyz="0.097841" ixz="0.0"/>
+    <origin xyz="0.42900000000000327 -0.07702054233668737 0.4385579778257891" rpy="0 0 0"/>
+    <mass value="11.56938089491454"/>
+    <inertia ixx="0.281385" iyy="1.751721" izz="1.497929" ixy="-0.0" iyz="0.033652" ixz="0.0"/>
   </inertial>
   <visual>
@@ -67,6 +67,6 @@
   <inertial>
     <origin xyz="-0.04012934689566563 -0.020235685434398354 -0.5125000000000013" rpy="0 0 0"/>
-    <mass value="22.428174832479133"/>
-    <inertia ixx="1.966316" iyy="1.974575" izz="0.013623" ixy="-5e-05" iyz="0.0" ixz="-0.0"/>
+    <mass value="7.714149305438682"/>
+    <inertia ixx="0.676312" iyy="0.679153" izz="0.004686" ixy="-1.7e-05" iyz="0.0" ixz="-0.0"/>
   </inertial>
   <visual>
@@ -86,7 +86,7 @@
 <link name="cabezal_1">
   <inertial>
-    <origin xyz="1.2055562844962009e-05 -0.074703758607254 0.074351694711558" rpy="0 0 0"/>
-    <mass value="5.246895030843086"/>
-    <inertia ixx="0.021135" iyy="0.008283" izz="0.018029" ixy="3e-06" iyz="0.004835" ixz="-1e-06"/>
+    <origin xyz="1.2055562844962009e-05 -0.07470375860725395 0.07435169471155806" rpy="0 0 0"/>
+    <mass value="0.735233698589477"/>
+    <inertia ixx="0.002962" iyy="0.001161" izz="0.002526" ixy="0.0" iyz="0.000677" ixz="-0.0"/>
   </inertial>
   <visual>
@@ -106,7 +106,7 @@
 <link name="Externo1_v1_1">
   <inertial>
-    <origin xyz="-1.124100812432971e-15 2.220446049250313e-16 -0.035297157702443877" rpy="0 0 0"/>
-    <mass value="3.103290090272312"/>
-    <inertia ixx="0.00441" iyy="0.004405" izz="0.008074" ixy="0.0" iyz="-0.0" ixz="0.0"/>
+    <origin xyz="-1.1310397063368782e-15 1.6653345369377348e-16 -0.035297157702443877" rpy="0 0 0"/>
+    <mass value="0.4348559362165023"/>
+    <inertia ixx="0.000618" iyy="0.000617" izz="0.001131" ixy="-0.0" iyz="-0.0" ixz="0.0"/>
   </inertial>
   <visual>
@@ -126,7 +126,7 @@
 <link name="cabezal_2.0_v1_1_1">
   <inertial>
-    <origin xyz="-1.9836844046515478e-05 0.00327884619901872 -0.05001506846643826" rpy="0 0 0"/>
-    <mass value="5.768314857333685"/>
-    <inertia ixx="0.020245" iyy="0.020069" izz="0.011543" ixy="0.0" iyz="0.000603" ixz="-4e-06"/>
+    <origin xyz="-1.9836844046515478e-05 0.00327884619901872 -0.050015068466438266" rpy="0 0 0"/>
+    <mass value="0.808298897205994"/>
+    <inertia ixx="0.002837" iyy="0.002812" izz="0.001617" ixy="0.0" iyz="8.5e-05" ixz="-1e-06"/>
   </inertial>
   <visual>
@@ -207,6 +207,6 @@
   <inertial>
     <origin xyz="-0.1070194860087463 0.004431382652601179 2.2922718924400787e-08" rpy="0 0 0"/>
-    <mass value="0.3818616414823265"/>
-    <inertia ixx="2.1e-05" iyy="0.00184" izz="0.001847" ixy="-8e-06" iyz="0.0" ixz="0.0"/>
+    <mass value="0.05350927460261899"/>
+    <inertia ixx="3e-06" iyy="0.000258" izz="0.000259" ixy="-1e-06" iyz="0.0" ixz="0.0"/>
   </inertial>
   <visual>
@@ -226,7 +226,7 @@
 <link name="Paleta_2_1">
   <inertial>
-    <origin xyz="0.10697797649072537 0.0053688772917466765 2.2922719278284376e-08" rpy="0 0 0"/>
-    <mass value="0.3818616414823265"/>
-    <inertia ixx="2.1e-05" iyy="0.00184" izz="0.001847" ixy="-8e-06" iyz="0.0" ixz="0.0"/>
+    <origin xyz="0.10697797649072537 0.005368877291746704 2.292271928522327e-08" rpy="0 0 0"/>
+    <mass value="0.05350927460261899"/>
+    <inertia ixx="3e-06" iyy="0.000258" izz="0.000259" ixy="-1e-06" iyz="0.0" ixz="0.0"/>
   </inertial>
   <visual>
@@ -247,6 +247,6 @@
   <inertial>
     <origin xyz="-0.02679441920888964 0.003882677544928881 -0.019023121817095687" rpy="0 0 0"/>
-    <mass value="1.1995109762545986"/>
-    <inertia ixx="0.003525" iyy="0.003481" izz="0.000292" ixy="0.0" iyz="-1e-06" ixz="-0.000204"/>
+    <mass value="0.1680843406216635"/>
+    <inertia ixx="0.000494" iyy="0.000488" izz="4.1e-05" ixy="0.0" iyz="-0.0" ixz="-2.9e-05"/>
   </inertial>
   <visual>
@@ -266,7 +266,7 @@
 <link name="Pala_DER_1">
   <inertial>
-    <origin xyz="0.026759728063148136 0.004117255172863543 -0.019023121817094694" rpy="0 0 0"/>
-    <mass value="1.1995109762545986"/>
-    <inertia ixx="0.003525" iyy="0.003481" izz="0.000292" ixy="0.0" iyz="1e-06" ixz="0.000204"/>
+    <origin xyz="0.02675972806314808 0.004117255172863543 -0.019023121817094694" rpy="0 0 0"/>
+    <mass value="0.1680843406216635"/>
+    <inertia ixx="0.000494" iyy="0.000488" izz="4.1e-05" ixy="0.0" iyz="0.0" ixz="2.9e-05"/>
   </inertial>
   <visual>
