Commit message: Actualiza las propiedades inerciales de los enlaces en robot_isaac.urdf para  la simulación en NVIDIA Isaac Sim.

File: src/robot_description/urdf/robot_isaac.urdf (robot description, URDF)
Before this commit: robot robot, 14 links, 13 joints
Links:
- link Externo1_v1_1: mass 3.103290090272312 -> 0.4348559362165023
- link Pala_DER_1: mass 1.1995109762545986 -> 0.1680843406216635
- link Pala_IZQ_1: mass 1.1995109762545986 -> 0.1680843406216635
- link Paleta_1_1: mass 0.3818616414823265 -> 0.05350927460261899
- link Paleta_2_1: mass 0.3818616414823265 -> 0.05350927460261899
- link base_link: mass 145.80079322670187 -> 50.148043530203196
- link cabezal_1: mass 5.246895030843086 -> 0.735233698589477
- link cabezal_2_0_v1_1_1: mass 5.768314857333685 -> 0.808298897205994
- link x_link_1: mass 33.63690371299227 -> 11.56938089491454
- link z_link_1: mass 22.428174832479133 -> 7.714149305438682
