Commit message: Cambios drasticos en la estructura y migracion a una version de gazebo mas actualizada

File: src/palletizer_description/urdf/materials.xacro (robot description, xacro)
@@ -1,4 +1,4 @@
 <?xml version="1.0" ?>
-<robot name="base_link_v_respaldo" xmlns:xacro="http://www.ros.org/wiki/xacro" >
+<robot name="palletizer" xmlns:xacro="http://www.ros.org/wiki/xacro" >
 <material name="silver">
   <color rgba="0.700 0.700 0.700 1.000"/>

File: src/palletizer_description/urdf/palletizer.xacro (robot description, xacro)
@@ -1,7 +1,12 @@
 <?xml version="1.0" ?>
-<robot name="base_link_v_respaldo" xmlns:xacro="http://www.ros.org/wiki/xacro">
-<xacro:include filename="$(find robot_description)/urdf/materials.xacro" />
-<xacro:include filename="$(find robot_description)/urdf/base_link_v_respaldo.trans" />
-<xacro:include filename="$(find robot_description)/urdf/base_link_v_respaldo.gazebo" />
+<robot name="palletizer" xmlns:xacro="http://www.ros.org/wiki/xacro">
+<xacro:include filename="$(find palletizer_description)/urdf/materials.xacro" />
+<xacro:include filename="$(find palletizer_description)/urdf/palletizer.gazebo" />
+<link name="world"/>
+<joint name="fixed_to_world" type="fixed">
+  <parent link="world"/>
+  <child link="base_link"/>
+  <origin xyz="0 0 0.01" rpy="0 0 0"/>
+</joint>
 <link name="base_link">
   <inertial>
@@ -13,14 +18,8 @@
     <origin xyz="0 0 0" rpy="0 0 0"/>
     <geometry>
-      <mesh filename="package://robot_description/meshes/base_link.stl" scale="0.001 0.001 0.001"/>
-    </geometry>
-    <material name="silver"/>
-  </visual>
-  <collision>
-    <origin xyz="0 0 0" rpy="0 0 0"/>
-    <geometry>
-      <mesh filename="package://robot_description/meshes/base_link.stl" scale="0.001 0.001 0.001"/>
-    </geometry>
-  </collision>
+      <mesh filename="package://palletizer_description/meshes/base_link.stl" scale="0.001 0.001 0.001"/>
+    </geometry>
+    <material name="silver"/>
+  </visual>
 </link>
 <link name="carro_x_der_1_1">
@@ -28,19 +27,13 @@
     <origin xyz="-0.0897790407869099 0.8137417184308351 0.09607295532194371" rpy="0 0 0"/>
     <mass value="1.2559999999999998"/>
-    <inertia ixx="0.00134" iyy="0.000735" izz="0.000735" ixy="0.0" iyz="-0.0" ixz="0.0"/>
+    <inertia ixx="0.01" iyy="0.01" izz="0.01" ixy="0.0" iyz="-0.0" ixz="0.0"/>
   </inertial>
   <visual>
     <origin xyz="-2.0 0.04 -0.72" rpy="0 0 0"/>
     <geometry>
-      <mesh filename="package://robot_description/meshes/carro_x_der_1_1.stl" scale="0.001 0.001 0.001"/>
-    </geometry>
-    <material name="silver"/>
-  </visual>
-  <collision>
-    <origin xyz="-2.0 0.04 -0.72" rpy="0 0 0"/>
-    <geometry>
-      <mesh filename="package://robot_description/meshes/carro_x_der_1_1.stl" scale="0.001 0.001 0.001"/>
-    </geometry>
-  </collision>
+      <mesh filename="package://palletizer_description/meshes/carro_x_der_1_1.stl" scale="0.001 0.001 0.001"/>
+    </geometry>
+    <material name="silver"/>
+  </visual>
 </link>
 <link name="carro_x_izq_1_1">
@@ -48,19 +41,13 @@
     <origin xyz="-0.06477904078692007 0.8137417184308272 0.09607295532194471" rpy="0 0 0"/>
     <mass value="1.2559999999999998"/>
-    <inertia ixx="0.00134" iyy="0.000735" izz="0.000735" ixy="0.0" iyz="-0.0" ixz="0.0"/>
+    <inertia ixx="0.01" iyy="0.01" izz="0.01" ixy="0.0" iyz="-0.0" ixz="0.0"/>
   </inertial>
   <visual>
     <origin xyz="0.0 0.04 -0.72" rpy="0 0 0"/>
     <geometry>
-      <mesh filename="package://robot_description/meshes/carro_x_izq_1_1.stl" scale="0.001 0.001 0.001"/>
-    </geometry>
-    <material name="silver"/>
-  </visual>
-  <collision>
-    <origin xyz="0.0 0.04 -0.72" rpy="0 0 0"/>
-    <geometry>
-      <mesh filename="package://robot_description/meshes/carro_x_izq_1_1.stl" scale="0.001 0.001 0.001"/>
-    </geometry>
-  </collision>
+      <mesh filename="package://palletizer_description/meshes/carro_x_izq_1_1.stl" scale="0.001 0.001 0.001"/>
+    </geometry>
+    <material name="silver"/>
+  </visual>
 </link>
 <link name="base_y_izq_1_1">
@@ -73,14 +60,8 @@
     <origin xyz="-0.025 0.04 -0.64" rpy="0 0 0"/>
     <geometry>
-      <mesh filename="package://robot_description/meshes/base_y_izq_1_1.stl" scale="0.001 0.001 0.001"/>
-    </geometry>
-    <material name="silver"/>
-  </visual>
-  <collision>
-    <origin xyz="-0.025 0.04 -0.64" rpy="0 0 0"/>
-    <geometry>
-      <mesh filename="package://robot_description/meshes/base_y_izq_1_1.stl" scale="0.001 0.001 0.001"/>
-    </geometry>
-  </collision>
+      <mesh filename="package://palletizer_description/meshes/base_y_izq_1_1.stl" scale="0.001 0.001 0.001"/>
+    </geometry>
+    <material name="silver"/>
+  </visual>
 </link>
 <link name="base_y_der_1_1">
@@ -93,14 +74,8 @@
     <origin xyz="-1.975 0.04 -0.64" rpy="0 0 0"/>
     <geometry>
-      <mesh filename="package://robot_description/meshes/base_y_der_1_1.stl" scale="0.001 0.001 0.001"/>
-    </geometry>
-    <material name="silver"/>
-  </visual>
-  <collision>
-    <origin xyz="-1.975 0.04 -0.64" rpy="0 0 0"/>
-    <geometry>
-      <mesh filename="package://robot_description/meshes/base_y_der_1_1.stl" scale="0.001 0.001 0.001"/>
-    </geometry>
-  </collision>
+      <mesh filename="package://palletizer_description/meshes/base_y_der_1_1.stl" scale="0.001 0.001 0.001"/>
+    </geometry>
+    <material name="silver"/>
+  </visual>
 </link>
 <link name="eje_carro_y_1_1">
@@ -113,14 +88,8 @@
     <origin xyz="0.052279 -0.733742 -1.456073" rpy="0 0 0"/>
     <geometry>
-      <mesh filename="package://robot_description/meshes/eje_carro_y_1_1.stl" scale="0.001 0.001 0.001"/>
-    </geometry>
-    <material name="silver"/>
-  </visual>
-  <collision>
-    <origin xyz="0.052279 -0.733742 -1.456073" rpy="0 0 0"/>
-    <geometry>
-      <mesh filename="package://robot_description/meshes/eje_carro_y_1_1.stl" scale="0.001 0.001 0.001"/>
-    </geometry>
-  </collision>
+      <mesh filename="package://palletizer_description/meshes/eje_carro_y_1_1.stl" scale="0.001 0.001 0.001"/>
+    </geometry>
+    <material name="silver"/>
+  </visual>
 </link>
 <link name="carro_y_1_1">
@@ -128,19 +97,13 @@
     <origin xyz="0.5213953273478066 -0.012500281569168936 -0.040000044678056845" rpy="0 0 0"/>
     <mass value="1.2559999999999998"/>
-    <inertia ixx="0.000735" iyy="0.00134" izz="0.000735" ixy="-0.0" iyz="0.0" ixz="0.0"/>
+    <inertia ixx="0.01" iyy="0.01" izz="0.01" ixy="-0.0" iyz="0.0" ixz="0.0"/>
   </inertial>
   <visual>
     <origin xyz="0.052279 -0.708742 -1.456073" rpy="0 0 0"/>
     <geometry>
-      <mesh filename="package://robot_description/meshes/carro_y_1_1.stl" scale="0.001 0.001 0.001"/>
-    </geometry>
-    <material name="silver"/>
-  </visual>
-  <collision>
-    <origin xyz="0.052279 -0.708742 -1.456073" rpy="0 0 0"/>
-    <geometry>
-      <mesh filename="package://robot_description/meshes/carro_y_1_1.stl" scale="0.001 0.001 0.001"/>
-    </geometry>
-  </collision>
+      <mesh filename="package://palletizer_description/meshes/carro_y_1_1.stl" scale="0.001 0.001 0.001"/>
+    </geometry>
+    <material name="silver"/>
+  </visual>
 </link>
 <link name="carro_z_1_1">
@@ -153,14 +116,8 @@
     <origin xyz="-0.509116 -0.683742 -1.456073" rpy="0 0 0"/>
     <geometry>
-      <mesh filename="package://robot_description/meshes/carro_z_1_1.stl" scale="0.001 0.001 0.001"/>
-    </geometry>
-    <material name="silver"/>
-  </visual>
-  <collision>
-    <origin xyz="-0.509116 -0.683742 -1.456073" rpy="0 0 0"/>
-    <geometry>
-      <mesh filename="package://robot_description/meshes/carro_z_1_1.stl" scale="0.001 0.001 0.001"/>
-    </geometry>
-  </collision>
+      <mesh filename="package://palletizer_description/meshes/carro_z_1_1.stl" scale="0.001 0.001 0.001"/>
+    </geometry>
+    <material name="silver"/>
+  </visual>
 </link>
 <link name="soporte_camara_1_1">
@@ -168,19 +125,13 @@
     <origin xyz="-0.03999967265219734 -0.012500281569165606 0.2300002666769576" rpy="0 0 0"/>
     <mass value="0.6279999999999999"/>
-    <inertia ixx="0.000116" iyy="0.000419" izz="0.000368" ixy="-0.0" iyz="0.0" ixz="-0.0"/>
+    <inertia ixx="0.01" iyy="0.01" izz="0.01" ixy="-0.0" iyz="0.0" ixz="-0.0"/>
   </inertial>
   <visual>
     <origin xyz="-0.509116 -0.658742 -0.591602" rpy="0 0 0"/>
     <geometry>
-      <mesh filename="package://robot_description/meshes/soporte_camara_1_1.stl" scale="0.001 0.001 0.001"/>
-    </geometry>
-    <material name="silver"/>
-  </visual>
-  <collision>
-    <origin xyz="-0.509116 -0.658742 -0.591602" rpy="0 0 0"/>
-    <geometry>
-      <mesh filename="package://robot_description/meshes/soporte_camara_1_1.stl" scale="0.001 0.001 0.001"/>
-    </geometry>
-  </collision>
+      <mesh filename="package://palletizer_description/meshes/soporte_camara_1_1.stl" scale="0.001 0.001 0.001"/>
+    </geometry>
+    <material name="silver"/>
+  </visual>
 </link>
 <link name="base_muneca_1_1">
@@ -188,19 +139,13 @@
     <origin xyz="-0.03999967265219412 -0.012500281569164162 0.01000026667695808" rpy="0 0 0"/>
     <mass value="0.6279999999999999"/>
-    <inertia ixx="0.000116" iyy="0.000419" izz="0.000368" ixy="0.0" iyz="0.0" ixz="-0.0"/>
+    <inertia ixx="0.01" iyy="0.01" izz="0.01" ixy="0.0" iyz="0.0" ixz="-0.0"/>
   </inertial>
   <visual>
     <origin xyz="-0.509116 -0.658742 -0.591602" rpy="0 0 0"/>
     <geometry>
-      <mesh filename="package://robot_description/meshes/base_muneca_1_1.stl" scale="0.001 0.001 0.001"/>
-    </geometry>
-    <material name="silver"/>
-  </visual>
-  <collision>
-    <origin xyz="-0.509116 -0.658742 -0.591602" rpy="0 0 0"/>
-    <geometry>
-      <mesh filename="package://robot_description/meshes/base_muneca_1_1.stl" scale="0.001 0.001 0.001"/>
-    </geometry>
-  </collision>
+      <mesh filename="package://palletizer_description/meshes/base_muneca_1_1.stl" scale="0.001 0.001 0.001"/>
+    </geometry>
+    <material name="silver"/>
+  </visual>
 </link>
 <link name="eje_muneca_izq_1">
@@ -208,19 +153,13 @@
     <origin xyz="-0.24311767265219475 0.27886571843083735 0.18938726667695815" rpy="0 0 0"/>
     <mass value="0.12330751165339957"/>
-    <inertia ixx="2e-06" iyy="0.000412" izz="0.000412" ixy="0.0" iyz="0.0" ixz="0.0"/>
+    <inertia ixx="0.01" iyy="0.01" izz="0.01" ixy="0.0" iyz="0.0" ixz="0.0"/>
   </inertial>
   <visual>
     <origin xyz="-0.652234 -0.367376 -0.402215" rpy="0 0 0"/>
     <geometry>
-      <mesh filename="package://robot_description/meshes/eje_muneca_izq_1.stl" scale="0.001 0.001 0.001"/>
-    </geometry>
-    <material name="silver"/>
-  </visual>
-  <collision>
-    <origin xyz="-0.652234 -0.367376 -0.402215" rpy="0 0 0"/>
-    <geometry>
-      <mesh filename="package://robot_description/meshes/eje_muneca_izq_1.stl" scale="0.001 0.001 0.001"/>
-    </geometry>
-  </collision>
+      <mesh filename="package://palletizer_description/meshes/eje_muneca_izq_1.stl" scale="0.001 0.001 0.001"/>
+    </geometry>
+    <material name="silver"/>
+  </visual>
 </link>
 <link name="eje_muneca_der_1_1">
@@ -228,19 +167,13 @@
     <origin xyz="-0.21709999379698341 0.2788657184308348 0.2493872666769576" rpy="0 0 0"/>
     <mass value="0.12330751165339962"/>
-    <inertia ixx="2e-06" iyy="0.000412" izz="0.000412" ixy="-0.0" iyz="-0.0" ixz="0.0"/>
+    <inertia ixx="0.01" iyy="0.01" izz="0.01" ixy="-0.0" iyz="-0.0" ixz="0.0"/>
   </inertial>
   <visual>
     <origin xyz="-0.732234 -0.367376 -0.362215" rpy="0 0 0"/>
     <geometry>
-      <mesh filename="package://robot_description/meshes/eje_muneca_der_1_1.stl" scale="0.001 0.001 0.001"/>
-    </geometry>
-    <material name="silver"/>
-  </visual>
-  <collision>
-    <origin xyz="-0.732234 -0.367376 -0.362215" rpy="0 0 0"/>
-    <geometry>
-      <mesh filename="package://robot_description/meshes/eje_muneca_der_1_1.stl" scale="0.001 0.001 0.001"/>
-    </geometry>
-  </collision>
+      <mesh filename="package://palletizer_description/meshes/eje_muneca_der_1_1.stl" scale="0.001 0.001 0.001"/>
+    </geometry>
+    <material name="silver"/>
+  </visual>
 </link>
 <link name="paleta_muneca_der_1">
@@ -253,14 +186,8 @@
     <origin xyz="-0.744269 -0.900107 -1.080989" rpy="0 0 0"/>
     <geometry>
-      <mesh filename="package://robot_description/meshes/paleta_muneca_der_1.stl" scale="0.001 0.001 0.001"/>
-    </geometry>
-    <material name="silver"/>
-  </visual>
-  <collision>
-    <origin xyz="-0.744269 -0.900107 -1.080989" rpy="0 0 0"/>
-    <geometry>
-      <mesh filename="package://robot_description/meshes/paleta_muneca_der_1.stl" scale="0.001 0.001 0.001"/>
-    </geometry>
-  </collision>
+      <mesh filename="package://palletizer_description/meshes/paleta_muneca_der_1.stl" scale="0.001 0.001 0.001"/>
+    </geometry>
+    <material name="silver"/>
+  </visual>
 </link>
 <link name="paleta_muneca_izq_1_1">
@@ -273,14 +200,8 @@
     <origin xyz="-0.207876 -0.392484 -1.069671" rpy="0 0 0"/>
     <geometry>
-      <mesh filename="package://robot_description/meshes/paleta_muneca_izq_1_1.stl" scale="0.001 0.001 0.001"/>
-    </geometry>
-    <material name="silver"/>
-  </visual>
-  <collision>
-    <origin xyz="-0.207876 -0.392484 -1.069671" rpy="0 0 0"/>
-    <geometry>
-      <mesh filename="package://robot_description/meshes/paleta_muneca_izq_1_1.stl" scale="0.001 0.001 0.001"/>
-    </geometry>
-  </collision>
+      <mesh filename="package://palletizer_description/meshes/paleta_muneca_izq_1_1.stl" scale="0.001 0.001 0.001"/>
+    </geometry>
+    <material name="silver"/>
+  </visual>
 </link>
 <link name="base_eje_x_izq_1_1">
@@ -293,14 +214,8 @@
     <origin xyz="0.0 0.04 -0.64" rpy="0 0 0"/>
     <geometry>
-      <mesh filename="package://robot_description/meshes/base_eje_x_izq_1_1.stl" scale="0.001 0.001 0.001"/>
-    </geometry>
-    <material name="silver"/>
-  </visual>
-  <collision>
-    <origin xyz="0.0 0.04 -0.64" rpy="0 0 0"/>
-    <geometry>
-      <mesh filename="package://robot_description/meshes/base_eje_x_izq_1_1.stl" scale="0.001 0.001 0.001"/>
-    </geometry>
-  </collision>
+      <mesh filename="package://palletizer_description/meshes/base_eje_x_izq_1_1.stl" scale="0.001 0.001 0.001"/>
+    </geometry>
+    <material name="silver"/>
+  </visual>
 </link>
 <link name="base_eje_x_der_1_1">
@@ -313,14 +228,8 @@
     <origin xyz="-2.04 0.04 -0.64" rpy="0 0 0"/>
     <geometry>
-      <mesh filename="package://robot_description/meshes/base_eje_x_der_1_1.stl" scale="0.001 0.001 0.001"/>
-    </geometry>
-    <material name="silver"/>
-  </visual>
-  <collision>
-    <origin xyz="-2.04 0.04 -0.64" rpy="0 0 0"/>
-    <geometry>
-      <mesh filename="package://robot_description/meshes/base_eje_x_der_1_1.stl" scale="0.001 0.001 0.001"/>
-    </geometry>
-  </collision>
+      <mesh filename="package://palletizer_description/meshes/base_eje_x_der_1_1.stl" scale="0.001 0.001 0.001"/>
+    </geometry>
+    <material name="silver"/>
+  </visual>
 </link>
 <joint name="Eje x" type="prismatic">
@@ -354,9 +263,4 @@
   <child link="eje_carro_y_1_1"/>
 </joint>
-<joint name="Rigida 8" type="fixed">
-  <origin xyz="-0.077279 0.773742 0.816073" rpy="0 0 0"/>
-  <parent link="base_y_izq_1_1"/>
-  <child link="eje_carro_y_1_1"/>
-</joint>
 <joint name="Eje y" type="prismatic">
   <origin xyz="0.0 -0.025 0.0" rpy="0 0 0"/>
@@ -418,3 +322,45 @@
   <child link="base_eje_x_der_1_1"/>
 </joint>
+<ros2_control name="IgnitionSystem" type="system">
+  <hardware>
+    <plugin>ign_ros2_control/IgnitionSystem</plugin>
+  </hardware>
+  <joint name="Eje x">
+    <command_interface name="position">
+      <param name="min">-0.40</param>
+      <param name="max">0.2</param>
+    </command_interface>
+    <state_interface name="position"/>
+    <state_interface name="velocity"/>
+  </joint>
+  <joint name="Eje y">
+    <command_interface name="position">
+      <param name="min">-0.75</param>
+      <param name="max">0.71</param>
+    </command_interface>
+    <state_interface name="position"/>
+    <state_interface name="velocity"/>
+  </joint>
+  <joint name="Eje z">
+    <command_interface name="position">
+      <param name="min">-1.0</param>
+      <param name="max">-0.05</param>
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