Commit message: feat: Update calibration and pick-and-place routines
- Renamed CalibradorManual to CalibradorPaletizador for clarity.
- Updated joint position limits in calibrador.py for improved configuration.
- Added PRUEBA_Z and PRUEBA_MUN variables for Z-axis and gripper control.
- Enhanced logging messages to provide clearer feedback on motor commands.
- Adjusted safe Z position in rutina_pick_and_place.py to align with new limits.
- Updated gripper closed position to reflect new calibration settings.

File: src/palletizer_description/urdf/materials.xacro (robot description, xacro)
@@ -2,5 +2,5 @@
 <robot name="palletizer" xmlns:xacro="http://www.ros.org/wiki/xacro" >
 <material name="silver">
-  <color rgba="0.700 0.700 0.700 1.000"/>
+  <color rgba="0.85 0.85 0.85 1.0"/>
 </material>
 </robot>

File: src/palletizer_description/urdf/palletizer.xacro (robot description, xacro)
@@ -1,366 +1,424 @@
 <?xml version="1.0" ?>
 <robot name="palletizer" xmlns:xacro="http://www.ros.org/wiki/xacro">
-<xacro:include filename="$(find palletizer_description)/urdf/materials.xacro" />
-<xacro:include filename="$(find palletizer_description)/urdf/palletizer.gazebo" />
-<link name="world"/>
-<joint name="fixed_to_world" type="fixed">
-  <parent link="world"/>
-  <child link="base_link"/>
-  <origin xyz="0 0 0.01" rpy="0 0 0"/>
-</joint>
-<link name="base_link">
-  <inertial>
-    <origin xyz="0.9227209592130785 0.5670413416556851 0.5148358419198835" rpy="0 0 0"/>
-    <mass value="97.4656"/>
-    <inertia ixx="16.747122" iyy="89.286245" izz="94.763561" ixy="0.0" iyz="-2.123132" ixz="0.0"/>
-  </inertial>
-  <visual>
-    <origin xyz="0 0 0" rpy="0 0 0"/>
-    <geometry>
-      <mesh filename="package://palletizer_description/meshes/base_link.stl" scale="0.001 0.001 0.001"/>
-    </geometry>
-    <material name="silver"/>
-  </visual>
-</link>
-<link name="carro_x_der_1_1">
-  <inertial>
-    <origin xyz="-0.0897790407869099 0.8137417184308351 0.09607295532194371" rpy="0 0 0"/>
-    <mass value="1.2559999999999998"/>
-    <inertia ixx="0.01" iyy="0.01" izz="0.01" ixy="0.0" iyz="-0.0" ixz="0.0"/>
-  </inertial>
-  <visual>
-    <origin xyz="-2.0 0.04 -0.72" rpy="0 0 0"/>
-    <geometry>
-      <mesh filename="package://palletizer_description/meshes/carro_x_der_1_1.stl" scale="0.001 0.001 0.001"/>
-    </geometry>
-    <material name="silver"/>
-  </visual>
-</link>
-<link name="carro_x_izq_1_1">
-  <inertial>
-    <origin xyz="-0.06477904078692007 0.8137417184308272 0.09607295532194471" rpy="0 0 0"/>
-    <mass value="1.2559999999999998"/>
-    <inertia ixx="0.01" iyy="0.01" izz="0.01" ixy="0.0" iyz="-0.0" ixz="0.0"/>
-  </inertial>
-  <visual>
-    <origin xyz="0.0 0.04 -0.72" rpy="0 0 0"/>
-    <geometry>
-      <mesh filename="package://palletizer_description/meshes/carro_x_izq_1_1.stl" scale="0.001 0.001 0.001"/>
-    </geometry>
-    <material name="silver"/>
-  </visual>
-</link>
-<link name="base_y_izq_1_1">
-  <inertial>
-    <origin xyz="-0.057279040786918894 0.8137417184308281 0.4760729553219435" rpy="0 0 0"/>
-    <mass value="17.081599999999998"/>
-    <inertia ixx="0.667321" iyy="0.660489" izz="0.011388" ixy="0.0" iyz="0.0" ixz="0.0"/>
-  </inertial>
-  <visual>
-    <origin xyz="-0.025 0.04 -0.64" rpy="0 0 0"/>
-    <geometry>
-      <mesh filename="package://palletizer_description/meshes/base_y_izq_1_1.stl" scale="0.001 0.001 0.001"/>
-    </geometry>
-    <material name="silver"/>
-  </visual>
-</link>
-<link name="base_y_der_1_1">
-  <inertial>
-    <origin xyz="-0.09727904078691152 0.8137417184308332 0.47607295532194416" rpy="0 0 0"/>
-    <mass value="17.081599999999998"/>
-    <inertia ixx="0.667321" iyy="0.660489" izz="0.011388" ixy="0.0" iyz="-0.0" ixz="-0.0"/>
-  </inertial>
-  <visual>
-    <origin xyz="-1.975 0.04 -0.64" rpy="0 0 0"/>
-    <geometry>
-      <mesh filename="package://palletizer_description/meshes/base_y_der_1_1.stl" scale="0.001 0.001 0.001"/>
-    </geometry>
-    <material name="silver"/>
-  </visual>
-</link>
-<link name="eje_carro_y_1_1">
-  <inertial>
-    <origin xyz="0.9749999592130977 -0.01250028156917038 -0.040000044678056845" rpy="0 0 0"/>
-    <mass value="30.614999999998826"/>
-    <inertia ixx="0.017923" iyy="9.717456" izz="9.702723" ixy="0.0" iyz="0.0" ixz="0.0"/>
-  </inertial>
-  <visual>
-    <origin xyz="0.052279 -0.733742 -1.456073" rpy="0 0 0"/>
-    <geometry>
-      <mesh filename="package://palletizer_description/meshes/eje_carro_y_1_1.stl" scale="0.001 0.001 0.001"/>
-    </geometry>
-    <material name="silver"/>
-  </visual>
-</link>
-<link name="carro_y_1_1">
-  <inertial>
-    <origin xyz="0.5213953273478066 -0.012500281569168936 -0.040000044678056845" rpy="0 0 0"/>
-    <mass value="1.2559999999999998"/>
-    <inertia ixx="0.01" iyy="0.01" izz="0.01" ixy="-0.0" iyz="0.0" ixz="0.0"/>
-  </inertial>
-  <visual>
-    <origin xyz="0.052279 -0.708742 -1.456073" rpy="0 0 0"/>
-    <geometry>
-      <mesh filename="package://palletizer_description/meshes/carro_y_1_1.stl" scale="0.001 0.001 0.001"/>
-    </geometry>
-    <material name="silver"/>
-  </visual>
-</link>
-<link name="carro_z_1_1">
-  <inertial>
-    <origin xyz="-0.039999672652193785 -0.012500281569168159 -0.22447073332304135" rpy="0 0 0"/>
-    <mass value="20.095999999999986"/>
-    <inertia ixx="2.744821" iyy="2.754492" izz="0.011765" ixy="0.0" iyz="0.0" ixz="0.0"/>
-  </inertial>
-  <visual>
-    <origin xyz="-0.509116 -0.683742 -1.456073" rpy="0 0 0"/>
-    <geometry>
-      <mesh filename="package://palletizer_description/meshes/carro_z_1_1.stl" scale="0.001 0.001 0.001"/>
-    </geometry>
-    <material name="silver"/>
-  </visual>
-</link>
-<link name="soporte_camara_1_1">
-  <inertial>
-    <origin xyz="-0.03999967265219734 -0.012500281569165606 0.2300002666769576" rpy="0 0 0"/>
-    <mass value="0.6279999999999999"/>
-    <inertia ixx="0.01" iyy="0.01" izz="0.01" ixy="-0.0" iyz="0.0" ixz="-0.0"/>
-  </inertial>
-  <visual>
-    <origin xyz="-0.509116 -0.658742 -0.591602" rpy="0 0 0"/>
-    <geometry>
-      <mesh filename="package://palletizer_description/meshes/soporte_camara_1_1.stl" scale="0.001 0.001 0.001"/>
-    </geometry>
-    <material name="silver"/>
-  </visual>
-</link>
-<link name="base_muneca_1_1">
-  <inertial>
-    <origin xyz="-0.03999967265219412 -0.012500281569164162 0.01000026667695808" rpy="0 0 0"/>
-    <mass value="0.6279999999999999"/>
-    <inertia ixx="0.01" iyy="0.01" izz="0.01" ixy="0.0" iyz="0.0" ixz="-0.0"/>
-  </inertial>
-  <visual>
-    <origin xyz="-0.509116 -0.658742 -0.591602" rpy="0 0 0"/>
-    <geometry>
-      <mesh filename="package://palletizer_description/meshes/base_muneca_1_1.stl" scale="0.001 0.001 0.001"/>
-    </geometry>
-    <material name="silver"/>
-  </visual>
-</link>
-<link name="eje_muneca_izq_1">
-  <inertial>
-    <origin xyz="-0.24311767265219475 0.27886571843083735 0.18938726667695815" rpy="0 0 0"/>
-    <mass value="0.12330751165339957"/>
-    <inertia ixx="0.01" iyy="0.01" izz="0.01" ixy="0.0" iyz="0.0" ixz="0.0"/>
-  </inertial>
-  <visual>
-    <origin xyz="-0.652234 -0.367376 -0.402215" rpy="0 0 0"/>
-    <geometry>
-      <mesh filename="package://palletizer_description/meshes/eje_muneca_izq_1.stl" scale="0.001 0.001 0.001"/>
-    </geometry>
-    <material name="silver"/>
-  </visual>
-</link>
-<link name="eje_muneca_der_1_1">
-  <inertial>
-    <origin xyz="-0.21709999379698341 0.2788657184308348 0.2493872666769576" rpy="0 0 0"/>
-    <mass value="0.12330751165339962"/>
-    <inertia ixx="0.01" iyy="0.01" izz="0.01" ixy="-0.0" iyz="-0.0" ixz="0.0"/>
-  </inertial>
-  <visual>
-    <origin xyz="-0.732234 -0.367376 -0.362215" rpy="0 0 0"/>
-    <geometry>
-      <mesh filename="package://palletizer_description/meshes/eje_muneca_der_1_1.stl" scale="0.001 0.001 0.001"/>
-    </geometry>
-    <material name="silver"/>
-  </visual>
-</link>
-<link name="paleta_muneca_der_1">
-  <inertial>
-    <origin xyz="-0.12163499379698262 -0.3438652815691654 -0.5143867333230419" rpy="0 0 0"/>
-    <mass value="2.590499999999999"/>
-    <inertia ixx="0.011247" iyy="0.002661" izz="0.008684" ixy="-0.0" iyz="0.0" ixz="0.0"/>
-  </inertial>
-  <visual>
-    <origin xyz="-0.744269 -0.900107 -1.080989" rpy="0 0 0"/>
-    <geometry>
-      <mesh filename="package://palletizer_description/meshes/paleta_muneca_der_1.stl" scale="0.001 0.001 0.001"/>
-    </geometry>
-    <material name="silver"/>
-  </visual>
-</link>
-<link name="paleta_muneca_izq_1_1">
-  <inertial>
-    <origin xyz="0.0937403273478058 0.16375771843083936 -0.5030687333230426" rpy="0 0 0"/>
-    <mass value="2.590499999999999"/>
-    <inertia ixx="0.011247" iyy="0.002661" izz="0.008684" ixy="-0.0" iyz="0.0" ixz="0.0"/>
-  </inertial>
-  <visual>
-    <origin xyz="-0.207876 -0.392484 -1.069671" rpy="0 0 0"/>
-    <geometry>
-      <mesh filename="package://palletizer_description/meshes/paleta_muneca_izq_1_1.stl" scale="0.001 0.001 0.001"/>
-    </geometry>
-    <material name="silver"/>
-  </visual>
-</link>
-<link name="base_eje_x_izq_1_1">
-  <inertial>
-    <origin xyz="-0.09727904078692015 0.4987939189752732 0.17607295532194467" rpy="0 0 0"/>
-    <mass value="22.1056"/>
-    <inertia ixx="1.438338" iyy="0.014737" izz="1.429495" ixy="0.0" iyz="0.0" ixz="0.0"/>
-  </inertial>
-  <visual>
-    <origin xyz="0.0 0.04 -0.64" rpy="0 0 0"/>
-    <geometry>
-      <mesh filename="package://palletizer_description/meshes/base_eje_x_izq_1_1.stl" scale="0.001 0.001 0.001"/>
-    </geometry>
-    <material name="silver"/>
-  </visual>
-</link>
-<link name="base_eje_x_der_1_1">
-  <inertial>
-    <origin xyz="-0.0972790407869224 0.498793918975273 0.17607295532194644" rpy="0 0 0"/>
-    <mass value="22.1056"/>
-    <inertia ixx="1.438338" iyy="0.014737" izz="1.429495" ixy="0.0" iyz="-0.0" ixz="0.0"/>
-  </inertial>
-  <visual>
-    <origin xyz="-2.04 0.04 -0.64" rpy="0 0 0"/>
-    <geometry>
-      <mesh filename="package://palletizer_description/meshes/base_eje_x_der_1_1.stl" scale="0.001 0.001 0.001"/>
-    </geometry>
-    <material name="silver"/>
-  </visual>
-</link>
-<joint name="Eje x" type="prismatic">
-  <origin xyz="-0.04 0.0 0.08" rpy="0 0 0"/>
-  <parent link="base_eje_x_der_1_1"/>
-  <child link="carro_x_der_1_1"/>
-  <axis xyz="-0.0 -1.0 0.0"/>
-  <limit upper="+0.2" lower="-0.40" effort="100" velocity="100"/>
-</joint>
-<joint name="Eje x copia" type="prismatic">
-  <origin xyz="0.0 0.0 0.08" rpy="0 0 0"/>
-  <parent link="base_eje_x_izq_1_1"/>
-  <child link="carro_x_izq_1_1"/>
-  <axis xyz="0.0 1.0 -0.0"/>
-  <limit upper="0.75" lower="0.2" effort="100" velocity="100"/>
-  <mimic joint="Eje x" multiplier="-1.0" offset="0.0"/>
-</joint>
-<joint name="Rigida 5" type="fixed">
-  <origin xyz="0.025 0.0 -0.08" rpy="0 0 0"/>
-  <parent link="carro_x_izq_1_1"/>
-  <child link="base_y_izq_1_1"/>
-</joint>
-<joint name="Rigida 6" type="fixed">
-  <origin xyz="-0.025 0.0 -0.08" rpy="0 0 0"/>
-  <parent link="carro_x_der_1_1"/>
-  <child link="base_y_der_1_1"/>
-</joint>
-<joint name="Rigida 7" type="fixed">
-  <origin xyz="-2.027279 0.773742 0.816073" rpy="0 0 0"/>
-  <parent link="base_y_der_1_1"/>
-  <child link="eje_carro_y_1_1"/>
-</joint>
-<joint name="Eje y" type="prismatic">
-  <origin xyz="0.0 -0.025 0.0" rpy="0 0 0"/>
-  <parent link="eje_carro_y_1_1"/>
-  <child link="carro_y_1_1"/>
-  <axis xyz="1.0 0.0 0.0"/>
-  <limit upper="0.71" lower="-0.75" effort="100" velocity="100"/>
-</joint>
-<joint name="Eje z" type="prismatic">
-  <origin xyz="0.561395 -0.025 0.0" rpy="0 0 0"/>
+  <xacro:include filename="$(find palletizer_description)/urdf/materials.xacro" />
+  <xacro:include filename="$(find palletizer_description)/urdf/palletizer.gazebo" />
+  <link name="world"/>
+  <joint name="fixed_to_world" type="fixed">
+    <parent link="world"/>
+    <child link="base_link"/>
+    <origin xyz="0 0 0.01" rpy="0 0 0"/>
+  </joint>
+  <link name="base_link">
+    <inertial>
+      <origin xyz="0.9227209592130785 0.5670413416556851 0.5148358419198835" rpy="0 0 0"/>
+      <mass value="97.4656"/>
+      <inertia ixx="16.747122" iyy="89.286245" izz="94.763561" ixy="0.0" iyz="-2.123132" ixz="0.0"/>
+    </inertial>
+    <visual>
+      <origin xyz="0 0 0" rpy="0 0 0"/>
+      <geometry>
+        <mesh filename="package://palletizer_description/meshes/base_link.stl" scale="0.001 0.001 0.001"/>
+      </geometry>
+      <material name="silver"/>
+    </visual>
+  </link>
+  <link name="base_eje_x_izq_1_1">
+    <inertial>
+      <origin xyz="-0.09727904078692015 0.4987939189752732 0.17607295532194467" rpy="0 0 0"/>
+      <mass value="22.1056"/>
+      <inertia ixx="1.438338" iyy="0.014737" izz="1.429495" ixy="0.0" iyz="0.0" ixz="0.0"/>
+    </inertial>
+    <visual>
+      <origin xyz="0.0 0.04 -0.64" rpy="0 0 0"/>
+      <geometry>
+        <mesh filename="package://palletizer_description/meshes/base_eje_x_izq_1_1.stl" scale="0.001 0.001 0.001"/>
+      </geometry>
+      <material name="silver"/>
+    </visual>
+  </link>
+  <link name="base_eje_x_der_1_1">
+    <inertial>
+      <origin xyz="-0.0972790407869224 0.498793918975273 0.17607295532194644" rpy="0 0 0"/>
+      <mass value="22.1056"/>
+      <inertia ixx="1.438338" iyy="0.014737" izz="1.429495" ixy="0.0" iyz="-0.0" ixz="0.0"/>
+    </inertial>
+    <visual>
+      <origin xyz="-2.04 0.04 -0.64" rpy="0 0 0"/>
+      <geometry>
+        <mesh filename="package://palletizer_description/meshes/base_eje_x_der_1_1.stl" scale="0.001 0.001 0.001"/>
+      </geometry>
+      <material name="silver"/>
+    </visual>
+  </link>
+  <joint name="Rigida 17" type="fixed">
+    <origin xyz="0.0 -0.04 0.64" rpy="0 0 0"/>
+    <parent link="base_link"/>
+    <child link="base_eje_x_izq_1_1"/>
+  </joint>
+  <joint name="Rigida 18" type="fixed">
+    <origin xyz="2.04 -0.04 0.64" rpy="0 0 0"/>
+    <parent link="base_link"/>
+    <child link="base_eje_x_der_1_1"/>
+  </joint>
+  <link name="carro_x_der_1_1">
+    <inertial>
+      <origin xyz="-0.0897790407869099 0.8137417184308351 0.09607295532194371" rpy="0 0 0"/>
+      <mass value="1.2559999999999998"/>
+      <inertia ixx="0.01" iyy="0.01" izz="0.01" ixy="0.0" iyz="-0.0" ixz="0.0"/>
+    </inertial>
+    <visual>
+      <origin xyz="-2.0 0.04 -0.72" rpy="0 0 0"/>
+      <geometry>
+        <mesh filename="package://palletizer_description/meshes/carro_x_der_1_1.stl" scale="0.001 0.001 0.001"/>
+      </geometry>
+      <material name="silver"/>
+    </visual>
+  </link>
+  <link name="carro_x_izq_1_1">
+    <inertial>
+      <origin xyz="-0.06477904078692007 0.8137417184308272 0.09607295532194471" rpy="0 0 0"/>
+      <mass value="1.2559999999999998"/>
+      <inertia ixx="0.01" iyy="0.01" izz="0.01" ixy="0.0" iyz="-0.0" ixz="0.0"/>
+    </inertial>
+    <visual>
+      <origin xyz="0.0 0.04 -0.72" rpy="0 0 0"/>
+      <geometry>
+        <mesh filename="package://palletizer_description/meshes/carro_x_izq_1_1.stl" scale="0.001 0.001 0.001"/>
+      </geometry>
+      <material name="silver"/>
+    </visual>
+  </link>
+  <joint name="Eje x" type="prismatic">
+    <origin xyz="-0.04 0.0 0.08" rpy="0 0 0"/>
+    <parent link="base_eje_x_der_1_1"/>
+    <child link="carro_x_der_1_1"/>
+    <axis xyz="0 1 0"/>
+    <limit lower="0.0" upper="0.6" effort="500" velocity="1.0"/>
+    <dynamics damping="10.0"/>
+  </joint>
+  <joint name="Eje x copia" type="prismatic">
+    <origin xyz="0.0 0.0 0.08" rpy="0 0 0"/>
+    <parent link="base_eje_x_izq_1_1"/>
+    <child link="carro_x_izq_1_1"/>
+    <axis xyz="0 1 0"/>
+    <limit lower="0.0" upper="0.6" effort="500" velocity="1.0"/>
+    <mimic joint="Eje x" multiplier="1.0" offset="0.0"/>
+    <dynamics damping="10.0"/>
+  </joint>
+  <link name="base_y_izq_1_1">
+    <inertial>
+      <origin xyz="-0.057279040786918894 0.8137417184308281 0.4760729553219435" rpy="0 0 0"/>
+      <mass value="17.081599999999998"/>
+      <inertia ixx="0.667321" iyy="0.660489" izz="0.011388" ixy="0.0" iyz="0.0" ixz="0.0"/>
+    </inertial>
+    <visual>
+      <origin xyz="-0.025 0.04 -0.64" rpy="0 0 0"/>
+      <geometry>
+        <mesh filename="package://palletizer_description/meshes/base_y_izq_1_1.stl" scale="0.001 0.001 0.001"/>
+      </geometry>
+      <material name="silver"/>
+    </visual>
+  </link>
+  <link name="base_y_der_1_1">
+    <inertial>
+      <origin xyz="-0.09727904078691152 0.8137417184308332 0.47607295532194416" rpy="0 0 0"/>
+      <mass value="17.081599999999998"/>
+      <inertia ixx="0.667321" iyy="0.660489" izz="0.011388" ixy="0.0" iyz="-0.0" ixz="-0.0"/>
+    </inertial>
+    <visual>
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