Commit message: fix : coliciones y movimiento, se agrego una gui para el movimeinto

File: src/palletizer_description/urdf/palletizer.xacro (robot description, xacro)
@@ -22,4 +22,10 @@
       <material name="silver"/>
     </visual>
+    <collision>
+      <origin xyz="0 0 0" rpy="0 0 0"/>
+      <geometry>
+        <mesh filename="package://palletizer_description/meshes/base_link.stl" scale="0.001 0.001 0.001"/>
+      </geometry>
+    </collision>
   </link>
   <link name="base_eje_x_izq_1_1">
@@ -36,4 +42,10 @@
       <material name="silver"/>
     </visual>
+    <collision>
+      <origin xyz="0.0 0.04 -0.64" rpy="0 0 0"/>
+      <geometry>
+        <mesh filename="package://palletizer_description/meshes/base_eje_x_izq_1_1.stl" scale="0.001 0.001 0.001"/>
+      </geometry>
+    </collision>
   </link>
   <link name="base_eje_x_der_1_1">
@@ -50,11 +62,17 @@
       <material name="silver"/>
     </visual>
-  </link>
-  <joint name="Rigida 17" type="fixed">
+    <collision>
+      <origin xyz="-2.04 0.04 -0.64" rpy="0 0 0"/>
+      <geometry>
+        <mesh filename="package://palletizer_description/meshes/base_eje_x_der_1_1.stl" scale="0.001 0.001 0.001"/>
+      </geometry>
+    </collision>
+  </link>
+  <joint name="rigida_17" type="fixed">
     <origin xyz="0.0 -0.04 0.64" rpy="0 0 0"/>
     <parent link="base_link"/>
     <child link="base_eje_x_izq_1_1"/>
   </joint>
-  <joint name="Rigida 18" type="fixed">
+  <joint name="rigida_18" type="fixed">
     <origin xyz="2.04 -0.04 0.64" rpy="0 0 0"/>
     <parent link="base_link"/>
@@ -74,4 +92,10 @@
       <material name="silver"/>
     </visual>
+    <collision>
+      <origin xyz="-2.0 0.04 -0.72" rpy="0 0 0"/>
+      <geometry>
+        <mesh filename="package://palletizer_description/meshes/carro_x_der_1_1.stl" scale="0.001 0.001 0.001"/>
+      </geometry>
+    </collision>
   </link>
   <link name="carro_x_izq_1_1">
@@ -88,6 +112,12 @@
       <material name="silver"/>
     </visual>
-  </link>
-  <joint name="Eje x" type="prismatic">
+    <collision>
+      <origin xyz="0.0 0.04 -0.72" rpy="0 0 0"/>
+      <geometry>
+        <mesh filename="package://palletizer_description/meshes/carro_x_izq_1_1.stl" scale="0.001 0.001 0.001"/>
+      </geometry>
+    </collision>
+  </link>
+  <joint name="eje_x" type="prismatic">
     <origin xyz="-0.04 0.0 0.08" rpy="0 0 0"/>
     <parent link="base_eje_x_der_1_1"/>
@@ -97,5 +127,5 @@
     <dynamics damping="10.0"/>
   </joint>
-  <joint name="Eje x copia" type="prismatic">
+  <joint name="eje_x_copia" type="prismatic">
     <origin xyz="0.0 0.0 0.08" rpy="0 0 0"/>
     <parent link="base_eje_x_izq_1_1"/>
@@ -103,5 +133,5 @@
     <axis xyz="0 1 0"/>
     <limit lower="0.0" upper="0.6" effort="500" velocity="1.0"/>
-    <mimic joint="Eje x" multiplier="1.0" offset="0.0"/>
+    <mimic joint="eje_x" multiplier="1.0" offset="0.0"/>
     <dynamics damping="10.0"/>
   </joint>
@@ -119,4 +149,10 @@
       <material name="silver"/>
     </visual>
+    <collision>
+      <origin xyz="-0.025 0.04 -0.64" rpy="0 0 0"/>
+      <geometry>
+        <mesh filename="package://palletizer_description/meshes/base_y_izq_1_1.stl" scale="0.001 0.001 0.001"/>
+      </geometry>
+    </collision>
   </link>
   <link name="base_y_der_1_1">
@@ -133,11 +169,17 @@
       <material name="silver"/>
     </visual>
-  </link>
-  <joint name="Rigida 5" type="fixed">
+    <collision>
+      <origin xyz="-1.975 0.04 -0.64" rpy="0 0 0"/>
+      <geometry>
+        <mesh filename="package://palletizer_description/meshes/base_y_der_1_1.stl" scale="0.001 0.001 0.001"/>
+      </geometry>
+    </collision>
+  </link>
+  <joint name="rigida_5" type="fixed">
     <origin xyz="0.025 0.0 -0.08" rpy="0 0 0"/>
     <parent link="carro_x_izq_1_1"/>
     <child link="base_y_izq_1_1"/>
   </joint>
-  <joint name="Rigida 6" type="fixed">
+  <joint name="rigida_6" type="fixed">
     <origin xyz="-0.025 0.0 -0.08" rpy="0 0 0"/>
     <parent link="carro_x_der_1_1"/>
@@ -157,6 +199,12 @@
       <material name="silver"/>
     </visual>
-  </link>
-  <joint name="Rigida 7" type="fixed">
+    <collision>
+      <origin xyz="0.052279 -0.733742 -1.456073" rpy="0 0 0"/>
+      <geometry>
+        <mesh filename="package://palletizer_description/meshes/eje_carro_y_1_1.stl" scale="0.001 0.001 0.001"/>
+      </geometry>
+    </collision>
+  </link>
+  <joint name="rigida_7" type="fixed">
     <origin xyz="-2.027279 0.773742 0.816073" rpy="0 0 0"/>
     <parent link="base_y_der_1_1"/>
@@ -176,6 +224,12 @@
       <material name="silver"/>
     </visual>
-  </link>
-  <joint name="Eje y" type="prismatic">
+    <collision>
+      <origin xyz="0.052279 -0.708742 -1.456073" rpy="0 0 0"/>
+      <geometry>
+        <mesh filename="package://palletizer_description/meshes/carro_y_1_1.stl" scale="0.001 0.001 0.001"/>
+      </geometry>
+    </collision>
+  </link>
+  <joint name="eje_y" type="prismatic">
     <origin xyz="0.0 -0.025 0.0" rpy="0 0 0"/>
     <parent link="eje_carro_y_1_1"/>
@@ -197,13 +251,18 @@
       <material name="silver"/>
     </visual>
-  </link>
-  <joint name="Eje z" type="prismatic">
-  <origin xyz="0.561395 -0.025 0.85" rpy="0 0 0"/>
-  <parent link="carro_y_1_1"/>
-  <child link="carro_z_1_1"/>
-  <axis xyz="0.0 0.0 -1.0"/>
-  <limit upper="0.0" lower="0.85" effort="2000" velocity="1.0"/>
-  <dynamics damping="1.0" friction="0.1"/>
-</joint>
+    <collision>
+      <origin xyz="-0.509116 -0.683742 -1.456073" rpy="0 0 0"/>
+      <geometry>
+        <mesh filename="package://palletizer_description/meshes/carro_z_1_1.stl" scale="0.001 0.001 0.001"/>
+      </geometry>
+    </collision>
+  </link>
+ <joint name="eje_z" type="prismatic">
+    <origin xyz="0.561395 -0.025 0.85" rpy="0 0 0"/>
+    <parent link="carro_y_1_1"/>
+    <child link="carro_z_1_1"/>
+    <axis xyz="0.0 0.0 1.0"/>
+    <limit lower="-0.90" upper="0.0" effort="2000" velocity="1.0"/>
+  </joint>
   <link name="base_muneca_1_1">
     <inertial>
@@ -219,6 +278,12 @@
       <material name="silver"/>
     </visual>
-  </link>
-  <joint name="Rigida 12" type="fixed">
+    <collision>
+      <origin xyz="-0.509116 -0.658742 -0.591602" rpy="0 0 0"/>
+      <geometry>
+        <mesh filename="package://palletizer_description/meshes/base_muneca_1_1.stl" scale="0.001 0.001 0.001"/>
+      </geometry>
+    </collision>
+  </link>
+  <joint name="rigida_12" type="fixed">
     <origin xyz="0.0 -0.025 -0.864471" rpy="0 0 0"/>
     <parent link="carro_z_1_1"/>
@@ -238,4 +303,10 @@
       <material name="silver"/>
     </visual>
+    <collision>
+      <origin xyz="-0.652234 -0.367376 -0.402215" rpy="0 0 0"/>
+      <geometry>
+        <mesh filename="package://palletizer_description/meshes/eje_muneca_izq_1.stl" scale="0.001 0.001 0.001"/>
+      </geometry>
+    </collision>
   </link>
   <link name="eje_muneca_der_1_1">
@@ -252,4 +323,10 @@
       <material name="silver"/>
     </visual>
+    <collision>
+      <origin xyz="-0.732234 -0.367376 -0.362215" rpy="0 0 0"/>
+      <geometry>
+        <mesh filename="package://palletizer_description/meshes/eje_muneca_der_1_1.stl" scale="0.001 0.001 0.001"/>
+      </geometry>
+    </collision>
   </link>
   <joint name="muneca" type="prismatic">
@@ -258,12 +335,12 @@
     <child link="eje_muneca_izq_1"/>
     <axis xyz="-1.0 0.0 0.0"/>
-    <limit upper="0.08" lower="-0.05" effort="100" velocity="1.0"/>
-  </joint>
-  <joint name="Corredera 14" type="prismatic">
+    <limit upper="0.08" lower="-0.05" effort="1000" velocity="1.0"/>
+  </joint>
+  <joint name="corredera_14" type="prismatic">
     <origin xyz="0.223118 -0.291366 -0.229387" rpy="0 0 0"/>
     <parent link="base_muneca_1_1"/>
     <child link="eje_muneca_der_1_1"/>
     <axis xyz="1.0 0.0 0.0"/>
-    <limit upper="0.08" lower="-0.05" effort="100" velocity="1.0"/>
+    <limit upper="0.08" lower="-0.05" effort="1000" velocity="1.0"/>
     <mimic joint="muneca" multiplier="1.0" offset="0.0"/>
   </joint>
@@ -281,4 +358,10 @@
       <material name="silver"/>
     </visual>
+    <collision>
+      <origin xyz="-0.744269 -0.900107 -1.080989" rpy="0 0 0"/>
+      <geometry>
+        <mesh filename="package://palletizer_description/meshes/paleta_muneca_der_1.stl" scale="0.001 0.001 0.001"/>
+      </geometry>
+    </collision>
   </link>
   <link name="paleta_muneca_izq_1_1">
@@ -295,11 +378,17 @@
       <material name="silver"/>
     </visual>
-  </link>
-  <joint name="Rigida 15" type="fixed">
+    <collision>
+      <origin xyz="-0.207876 -0.392484 -1.069671" rpy="0 0 0"/>
+      <geometry>
+        <mesh filename="package://palletizer_description/meshes/paleta_muneca_izq_1_1.stl" scale="0.001 0.001 0.001"/>
+      </geometry>
+    </collision>
+  </link>
+  <joint name="rigida_15" type="fixed">
     <origin xyz="0.012035 0.532731 0.718774" rpy="0 0 0"/>
     <parent link="eje_muneca_der_1_1"/>
     <child link="paleta_muneca_der_1"/>
   </joint>
-  <joint name="Rigida 16" type="fixed">
+  <joint name="rigida_16" type="fixed">
     <origin xyz="-0.444358 0.025108 0.667456" rpy="0 0 0"/>
     <parent link="eje_muneca_izq_1"/>
@@ -319,6 +408,12 @@
       <material name="silver"/>
     </visual>
-  </link>
-  <joint name="Rigida 11" type="fixed">
+    <collision>
+      <origin xyz="-0.509116 -0.658742 -0.591602" rpy="0 0 0"/>
+      <geometry>
+        <mesh filename="package://palletizer_description/meshes/soporte_camara_1_1.stl" scale="0.001 0.001 0.001"/>
+      </geometry>
+    </collision>
+  </link>
+  <joint name="rigida_11" type="fixed">
     <origin xyz="0.0 -0.025 -0.864471" rpy="0 0 0"/>
     <parent link="carro_z_1_1"/>
@@ -338,4 +433,10 @@
       <material name="silver"/>
     </visual>
+    <collision>
+      <origin xyz="0 0 0" rpy="0 0 0"/>
+      <geometry>
+        <box size="0.05 0.05 0.05"/>
+      </geometry>
+    </collision>
   </link>
   <joint name="camera_joint" type="fixed">
@@ -344,4 +445,16 @@
     <child link="camera_link"/>
   </joint>
+  <gazebo reference="paleta_muneca_der_1">
+    <mu1>100.0</mu1>
+    <mu2>100.0</mu2>
+    <kp>1000000.0</kp>
+    <kd>1.0</kd>
+  </gazebo>
+  <gazebo reference="paleta_muneca_izq_1_1">
+    <mu1>100.0</mu1>
+    <mu2>100.0</mu2>
+    <kp>1000000.0</kp>
+    <kd>1.0</kd>
+  </gazebo>
   <gazebo reference="camera_link">
     <sensor name="camera_sensor" type="camera">
@@ -370,5 +483,5 @@
       <plugin>gz_ros2_control/GazeboSimSystem</plugin>
     </hardware>
-    <joint name="Eje x">
+    <joint name="eje_x">
       <command_interface name="position">
         <param name="min">0.0</param>
@@ -378,6 +491,6 @@
       <state_interface name="velocity"/>
     </joint>
-    <joint name="Eje x copia">
-      <param name="mimic">Eje x</param>
+    <joint name="eje_x_copia">
+      <param name="mimic">eje_x</param>
       <param name="multiplier">1.0</param>
       <command_interface name="position"/>
@@ -385,5 +498,5 @@
       <state_interface name="velocity"/>
     </joint>
-    <joint name="Eje y">
+    <joint name="eje_y">
       <command_interface name="position">
         <param name="min">-0.75</param>
@@ -393,8 +506,8 @@
       <state_interface name="velocity"/>
     </joint>
-    <joint name="Eje z">
+    <joint name="eje_z">
       <command_interface name="position">
-        <param name="min">0.0</param>
-        <param name="max">0.85</param>
+        <param name="min">-0.90</param>
+        <param name="max">0.0</param>
       </command_interface>
       <state_interface name="position"/>
@@ -409,5 +522,5 @@
       <state_interface name="velocity"/>
     </joint>
-    <joint name="Corredera 14">
+    <joint name="corredera_14">
       <param name="mimic">muneca</param>
       <param name="multiplier">1.0</param>
@@ -422,3 +535,30 @@
     </plugin>
   </gazebo>
+  <gazebo reference="carro_z_1_1">
+    <gravity>false</gravity>
+  </gazebo>
+  <gazebo reference="carro_z_1_1">
+    <gravity>false</gravity>
+  </gazebo>
+  <gazebo reference="base_muneca_1_1">
+    <gravity>false</gravity>
+  </gazebo>
+  <gazebo reference="eje_muneca_izq_1">
+    <gravity>false</gravity>
+  </gazebo>
+  <gazebo reference="eje_muneca_der_1_1">
+    <gravity>false</gravity>
+  </gazebo>
+  <gazebo reference="paleta_muneca_der_1">
+    <gravity>false</gravity>
+  </gazebo>
+  <gazebo reference="paleta_muneca_izq_1_1">
+    <gravity>false</gravity>
+  </gazebo>
+  <gazebo reference="soporte_camara_1_1">
+    <gravity>false</gravity>
+  </gazebo>
+  <gazebo reference="camera_link">
+    <gravity>false</gravity>
+  </gazebo>
 </robot>
