Commit message: Rename package intento_3_description to robot_paletizador and update references

File: src/robot_paletizador/urdf/materials.xacro (robot description, xacro)
@@ -1,4 +1,4 @@
 <?xml version="1.0" ?>
-<robot name="intento_3" xmlns:xacro="http://www.ros.org/wiki/xacro" >
+<robot name="robot_paletizador" xmlns:xacro="http://www.ros.org/wiki/xacro" >
 <material name="silver">
   <color rgba="0.700 0.700 0.700 1.000"/>

File: src/robot_paletizador/urdf/robot_paletizador.xacro (robot description, xacro)
@@ -1,7 +1,7 @@
 <?xml version="1.0" ?>
-<robot name="intento_3" xmlns:xacro="http://www.ros.org/wiki/xacro">
-<xacro:include filename="$(find intento_3_description)/urdf/materials.xacro" />
-<xacro:include filename="$(find intento_3_description)/urdf/intento_3.trans" />
-<xacro:include filename="$(find intento_3_description)/urdf/intento_3.gazebo" />
+<robot name="robot_paletizador" xmlns:xacro="http://www.ros.org/wiki/xacro">
+<xacro:include filename="$(find robot_paletizador)/urdf/materials.xacro" />
+<xacro:include filename="$(find robot_paletizador)/urdf/robot_paletizador.trans" />
+<xacro:include filename="$(find robot_paletizador)/urdf/robot_paletizador.gazebo" />
 <link name="base_link">
   <inertial>
@@ -13,5 +13,5 @@
     <origin xyz="0 0 0" rpy="0 0 0"/>
     <geometry>
-      <mesh filename="package://intento_3_description/meshes/base_link.stl" scale="0.001 0.001 0.001"/>
+      <mesh filename="package://robot_paletizador/meshes/base_link.stl" scale="0.001 0.001 0.001"/>
     </geometry>
     <material name="silver"/>
@@ -20,5 +20,5 @@
     <origin xyz="0 0 0" rpy="0 0 0"/>
     <geometry>
-      <mesh filename="package://intento_3_description/meshes/base_link.stl" scale="0.001 0.001 0.001"/>
+      <mesh filename="package://robot_paletizador/meshes/base_link.stl" scale="0.001 0.001 0.001"/>
     </geometry>
   </collision>
@@ -33,5 +33,5 @@
     <origin xyz="-0.15521 0.53479 -0.42" rpy="0 0 0"/>
     <geometry>
-      <mesh filename="package://intento_3_description/meshes/eje_x_link_1.stl" scale="0.001 0.001 0.001"/>
+      <mesh filename="package://robot_paletizador/meshes/eje_x_link_1.stl" scale="0.001 0.001 0.001"/>
     </geometry>
     <material name="silver"/>
@@ -40,5 +40,5 @@
     <origin xyz="-0.15521 0.53479 -0.42" rpy="0 0 0"/>
     <geometry>
-      <mesh filename="package://intento_3_description/meshes/eje_x_link_1.stl" scale="0.001 0.001 0.001"/>
+      <mesh filename="package://robot_paletizador/meshes/eje_x_link_1.stl" scale="0.001 0.001 0.001"/>
     </geometry>
   </collision>
@@ -53,5 +53,5 @@
     <origin xyz="-0.23521 -0.15521 -0.9" rpy="0 0 0"/>
     <geometry>
-      <mesh filename="package://intento_3_description/meshes/eje_y_link_1.stl" scale="0.001 0.001 0.001"/>
+      <mesh filename="package://robot_paletizador/meshes/eje_y_link_1.stl" scale="0.001 0.001 0.001"/>
     </geometry>
     <material name="silver"/>
@@ -60,5 +60,5 @@
     <origin xyz="-0.23521 -0.15521 -0.9" rpy="0 0 0"/>
     <geometry>
-      <mesh filename="package://intento_3_description/meshes/eje_y_link_1.stl" scale="0.001 0.001 0.001"/>
+      <mesh filename="package://robot_paletizador/meshes/eje_y_link_1.stl" scale="0.001 0.001 0.001"/>
     </geometry>
   </collision>
@@ -73,5 +73,5 @@
     <origin xyz="-0.26021 -0.15521 -0.9" rpy="0 0 0"/>
     <geometry>
-      <mesh filename="package://intento_3_description/meshes/eje_z_link_1.stl" scale="0.001 0.001 0.001"/>
+      <mesh filename="package://robot_paletizador/meshes/eje_z_link_1.stl" scale="0.001 0.001 0.001"/>
     </geometry>
     <material name="silver"/>
@@ -80,5 +80,5 @@
     <origin xyz="-0.26021 -0.15521 -0.9" rpy="0 0 0"/>
     <geometry>
-      <mesh filename="package://intento_3_description/meshes/eje_z_link_1.stl" scale="0.001 0.001 0.001"/>
+      <mesh filename="package://robot_paletizador/meshes/eje_z_link_1.stl" scale="0.001 0.001 0.001"/>
     </geometry>
   </collision>
@@ -93,5 +93,5 @@
     <origin xyz="-0.27271 -0.15521 -0.3" rpy="0 0 0"/>
     <geometry>
-      <mesh filename="package://intento_3_description/meshes/r_link_1.stl" scale="0.001 0.001 0.001"/>
+      <mesh filename="package://robot_paletizador/meshes/r_link_1.stl" scale="0.001 0.001 0.001"/>
     </geometry>
     <material name="silver"/>
@@ -100,5 +100,5 @@
     <origin xyz="-0.27271 -0.15521 -0.3" rpy="0 0 0"/>
     <geometry>
-      <mesh filename="package://intento_3_description/meshes/r_link_1.stl" scale="0.001 0.001 0.001"/>
+      <mesh filename="package://robot_paletizador/meshes/r_link_1.stl" scale="0.001 0.001 0.001"/>
     </geometry>
   </collision>
@@ -113,5 +113,5 @@
     <origin xyz="-0.545421 -0.315421 -0.59" rpy="0 0 0"/>
     <geometry>
-      <mesh filename="package://intento_3_description/meshes/griper_der_link_1.stl" scale="0.001 0.001 0.001"/>
+      <mesh filename="package://robot_paletizador/meshes/griper_der_link_1.stl" scale="0.001 0.001 0.001"/>
     </geometry>
     <material name="silver"/>
@@ -120,5 +120,5 @@
     <origin xyz="-0.545421 -0.315421 -0.59" rpy="0 0 0"/>
     <geometry>
-      <mesh filename="package://intento_3_description/meshes/griper_der_link_1.stl" scale="0.001 0.001 0.001"/>
+      <mesh filename="package://robot_paletizador/meshes/griper_der_link_1.stl" scale="0.001 0.001 0.001"/>
     </geometry>
   </collision>
@@ -133,5 +133,5 @@
     <origin xyz="-0.545421 -0.305421 -0.57" rpy="0 0 0"/>
     <geometry>
-      <mesh filename="package://intento_3_description/meshes/griper_izq_link_1.stl" scale="0.001 0.001 0.001"/>
+      <mesh filename="package://robot_paletizador/meshes/griper_izq_link_1.stl" scale="0.001 0.001 0.001"/>
     </geometry>
     <material name="silver"/>
@@ -140,5 +140,5 @@
     <origin xyz="-0.545421 -0.305421 -0.57" rpy="0 0 0"/>
     <geometry>
-      <mesh filename="package://intento_3_description/meshes/griper_izq_link_1.stl" scale="0.001 0.001 0.001"/>
+      <mesh filename="package://robot_paletizador/meshes/griper_izq_link_1.stl" scale="0.001 0.001 0.001"/>
     </geometry>
   </collision>
