Commit message: Desplazamiento de los joint que estaban corridos del proeycto robot_ensable_descripotion en los .xacro .urdf, .gazebo

File: src/robot_ensamble_description/urdf/robot_ensamble.xacro (robot description, xacro)
@@ -1,7 +1,12 @@
 <?xml version="1.0" ?>
 <robot name="robot_ensamble" xmlns:xacro="http://www.ros.org/wiki/xacro">
-<xacro:include filename="$(find robot_ensamble_description)/urdf/materials.xacro" />
-<xacro:include filename="$(find robot_ensamble_description)/urdf/robot_ensamble.trans" />
-<xacro:include filename="$(find robot_ensamble_description)/urdf/robot_ensamble.gazebo" />
+<!-- ROS usa package://; la exportacion para Isaac usa ../meshes/. -->
+<xacro:arg name="mesh_prefix" default="package://robot_ensamble_description/meshes/" />
+<xacro:arg name="include_ros_extensions" default="true" />
+<xacro:include filename="materials.xacro" />
+<xacro:if value="$(arg include_ros_extensions)">
+  <xacro:include filename="robot_ensamble.trans" />
+  <xacro:include filename="robot_ensamble.gazebo" />
+</xacro:if>
 <link name="base_link">
   <inertial>
@@ -13,5 +18,5 @@
     <origin xyz="0 0 0" rpy="0 0 0"/>
     <geometry>
-      <mesh filename="file://$(find robot_ensamble_description)/meshes/base_link.stl" scale="0.001 0.001 0.001"/>
+      <mesh filename="$(arg mesh_prefix)base_link.stl" scale="0.001 0.001 0.001"/>
     </geometry>
     <material name="silver"/>
@@ -20,5 +25,5 @@
     <origin xyz="0 0 0" rpy="0 0 0"/>
     <geometry>
-      <mesh filename="file://$(find robot_ensamble_description)/meshes/base_link.stl" scale="0.001 0.001 0.001"/>
+      <mesh filename="$(arg mesh_prefix)base_link.stl" scale="0.001 0.001 0.001"/>
     </geometry>
   </collision>
@@ -33,5 +38,5 @@
     <origin xyz="0.02001 -0.03 -0.6215" rpy="0 0 0"/>
     <geometry>
-      <mesh filename="file://$(find robot_ensamble_description)/meshes/x_link_1.stl" scale="0.001 0.001 0.001"/>
+      <mesh filename="$(arg mesh_prefix)x_link_1.stl" scale="0.001 0.001 0.001"/>
     </geometry>
     <material name="silver"/>
@@ -40,5 +45,5 @@
     <origin xyz="0.02001 -0.03 -0.6215" rpy="0 0 0"/>
     <geometry>
-      <mesh filename="file://$(find robot_ensamble_description)/meshes/x_link_1.stl" scale="0.001 0.001 0.001"/>
+      <mesh filename="$(arg mesh_prefix)x_link_1.stl" scale="0.001 0.001 0.001"/>
     </geometry>
   </collision>
@@ -53,5 +58,5 @@
     <origin xyz="-0.10999 0.0325 -1.023" rpy="0 0 0"/>
     <geometry>
-      <mesh filename="file://$(find robot_ensamble_description)/meshes/y_link_1.stl" scale="0.001 0.001 0.001"/>
+      <mesh filename="$(arg mesh_prefix)y_link_1.stl" scale="0.001 0.001 0.001"/>
     </geometry>
     <material name="silver"/>
@@ -60,5 +65,5 @@
     <origin xyz="-0.10999 0.0325 -1.023" rpy="0 0 0"/>
     <geometry>
-      <mesh filename="file://$(find robot_ensamble_description)/meshes/y_link_1.stl" scale="0.001 0.001 0.001"/>
+      <mesh filename="$(arg mesh_prefix)y_link_1.stl" scale="0.001 0.001 0.001"/>
     </geometry>
   </collision>
@@ -73,5 +78,5 @@
     <origin xyz="-0.11499 0.0325 -1.023" rpy="0 0 0"/>
     <geometry>
-      <mesh filename="file://$(find robot_ensamble_description)/meshes/z_link_1.stl" scale="0.001 0.001 0.001"/>
+      <mesh filename="$(arg mesh_prefix)z_link_1.stl" scale="0.001 0.001 0.001"/>
     </geometry>
     <material name="silver"/>
@@ -80,5 +85,5 @@
     <origin xyz="-0.11499 0.0325 -1.023" rpy="0 0 0"/>
     <geometry>
-      <mesh filename="file://$(find robot_ensamble_description)/meshes/z_link_1.stl" scale="0.001 0.001 0.001"/>
+      <mesh filename="$(arg mesh_prefix)z_link_1.stl" scale="0.001 0.001 0.001"/>
     </geometry>
   </collision>
@@ -93,5 +98,5 @@
     <origin xyz="-0.15499 -0.006 -1.023" rpy="0 0 0"/>
     <geometry>
-      <mesh filename="file://$(find robot_ensamble_description)/meshes/complemento_cabezal_1.stl" scale="0.001 0.001 0.001"/>
+      <mesh filename="$(arg mesh_prefix)complemento_cabezal_1.stl" scale="0.001 0.001 0.001"/>
     </geometry>
     <material name="silver"/>
@@ -100,5 +105,5 @@
     <origin xyz="-0.15499 -0.006 -1.023" rpy="0 0 0"/>
     <geometry>
-      <mesh filename="file://$(find robot_ensamble_description)/meshes/complemento_cabezal_1.stl" scale="0.001 0.001 0.001"/>
+      <mesh filename="$(arg mesh_prefix)complemento_cabezal_1.stl" scale="0.001 0.001 0.001"/>
     </geometry>
   </collision>
@@ -113,5 +118,5 @@
     <origin xyz="-0.16099 -0.006 -1.023" rpy="0 0 0"/>
     <geometry>
-      <mesh filename="file://$(find robot_ensamble_description)/meshes/robot_cabezal_1.stl" scale="0.001 0.001 0.001"/>
+      <mesh filename="$(arg mesh_prefix)robot_cabezal_1.stl" scale="0.001 0.001 0.001"/>
     </geometry>
     <material name="silver"/>
@@ -120,5 +125,5 @@
     <origin xyz="-0.16099 -0.006 -1.023" rpy="0 0 0"/>
     <geometry>
-      <mesh filename="file://$(find robot_ensamble_description)/meshes/robot_cabezal_1.stl" scale="0.001 0.001 0.001"/>
+      <mesh filename="$(arg mesh_prefix)robot_cabezal_1.stl" scale="0.001 0.001 0.001"/>
     </geometry>
   </collision>
@@ -133,5 +138,5 @@
     <origin xyz="-0.21099 -0.006 -1.0375" rpy="0 0 0"/>
     <geometry>
-      <mesh filename="file://$(find robot_ensamble_description)/meshes/acople_cabeza_1.stl" scale="0.001 0.001 0.001"/>
+      <mesh filename="$(arg mesh_prefix)acople_cabeza_1.stl" scale="0.001 0.001 0.001"/>
     </geometry>
     <material name="silver"/>
@@ -140,5 +145,5 @@
     <origin xyz="-0.21099 -0.006 -1.0375" rpy="0 0 0"/>
     <geometry>
-      <mesh filename="file://$(find robot_ensamble_description)/meshes/acople_cabeza_1.stl" scale="0.001 0.001 0.001"/>
+      <mesh filename="$(arg mesh_prefix)acople_cabeza_1.stl" scale="0.001 0.001 0.001"/>
     </geometry>
   </collision>
@@ -153,5 +158,5 @@
     <origin xyz="-0.21099 -0.006 -0.988" rpy="0 0 0"/>
     <geometry>
-      <mesh filename="file://$(find robot_ensamble_description)/meshes/cabezal_inferior_1.stl" scale="0.001 0.001 0.001"/>
+      <mesh filename="$(arg mesh_prefix)cabezal_inferior_1.stl" scale="0.001 0.001 0.001"/>
     </geometry>
     <material name="silver"/>
@@ -160,5 +165,5 @@
     <origin xyz="-0.21099 -0.006 -0.988" rpy="0 0 0"/>
     <geometry>
-      <mesh filename="file://$(find robot_ensamble_description)/meshes/cabezal_inferior_1.stl" scale="0.001 0.001 0.001"/>
+      <mesh filename="$(arg mesh_prefix)cabezal_inferior_1.stl" scale="0.001 0.001 0.001"/>
     </geometry>
   </collision>
@@ -173,5 +178,5 @@
     <origin xyz="-0.190512 -0.00091 -0.8725" rpy="0 0 0"/>
     <geometry>
-      <mesh filename="file://$(find robot_ensamble_description)/meshes/servo_mg996R_1.stl" scale="0.001 0.001 0.001"/>
+      <mesh filename="$(arg mesh_prefix)servo_mg996R_1.stl" scale="0.001 0.001 0.001"/>
     </geometry>
     <material name="silver"/>
@@ -180,5 +185,5 @@
     <origin xyz="-0.190512 -0.00091 -0.8725" rpy="0 0 0"/>
     <geometry>
-      <mesh filename="file://$(find robot_ensamble_description)/meshes/servo_mg996R_1.stl" scale="0.001 0.001 0.001"/>
+      <mesh filename="$(arg mesh_prefix)servo_mg996R_1.stl" scale="0.001 0.001 0.001"/>
     </geometry>
   </collision>
@@ -188,10 +193,12 @@
     <origin xyz="0.0031874891212040346 1.4413294836576607e-05 -1.4432899320127035e-15" rpy="0 0 0"/>
     <mass value="0.005099610361289279"/>
-    <inertia ixx="0.0" iyy="0.0" izz="0.0" ixy="0.0" iyz="0.0" ixz="0.0"/>
+    <!-- Estimacion por integracion del STL a escala metrica y densidad uniforme,
+         con la masa y el origen inercial CAD originales; unidades kg*m^2. -->
+    <inertia ixx="2.4043692089e-07" iyy="1.2530990918e-07" izz="1.2530779899e-07" ixy="5.0477842017e-10" iyz="-5.3076659018e-16" ixz="2.4812060723e-16"/>
   </inertial>
   <visual>
     <origin xyz="-0.20249 -0.005962 -0.907" rpy="0 0 0"/>
     <geometry>
-      <mesh filename="file://$(find robot_ensamble_description)/meshes/horn_Servo_1.stl" scale="0.001 0.001 0.001"/>
+      <mesh filename="$(arg mesh_prefix)horn_Servo_1.stl" scale="0.001 0.001 0.001"/>
     </geometry>
     <material name="silver"/>
@@ -200,5 +207,5 @@
     <origin xyz="-0.20249 -0.005962 -0.907" rpy="0 0 0"/>
     <geometry>
-      <mesh filename="file://$(find robot_ensamble_description)/meshes/horn_Servo_1.stl" scale="0.001 0.001 0.001"/>
+      <mesh filename="$(arg mesh_prefix)horn_Servo_1.stl" scale="0.001 0.001 0.001"/>
     </geometry>
   </collision>
@@ -213,5 +220,5 @@
     <origin xyz="-0.20699 -0.005982 -0.907" rpy="0 0 0"/>
     <geometry>
-      <mesh filename="file://$(find robot_ensamble_description)/meshes/acople_palas_1.stl" scale="0.001 0.001 0.001"/>
+      <mesh filename="$(arg mesh_prefix)acople_palas_1.stl" scale="0.001 0.001 0.001"/>
     </geometry>
     <material name="silver"/>
@@ -220,5 +227,5 @@
     <origin xyz="-0.20699 -0.005982 -0.907" rpy="0 0 0"/>
     <geometry>
-      <mesh filename="file://$(find robot_ensamble_description)/meshes/acople_palas_1.stl" scale="0.001 0.001 0.001"/>
+      <mesh filename="$(arg mesh_prefix)acople_palas_1.stl" scale="0.001 0.001 0.001"/>
     </geometry>
   </collision>
@@ -233,5 +240,5 @@
     <origin xyz="-0.2041 0.019031 -0.907" rpy="0 0 0"/>
     <geometry>
-      <mesh filename="file://$(find robot_ensamble_description)/meshes/Paleta_grid_1_1.stl" scale="0.001 0.001 0.001"/>
+      <mesh filename="$(arg mesh_prefix)Paleta_grid_1_1.stl" scale="0.001 0.001 0.001"/>
     </geometry>
     <material name="silver"/>
@@ -240,5 +247,5 @@
     <origin xyz="-0.2041 0.019031 -0.907" rpy="0 0 0"/>
     <geometry>
-      <mesh filename="file://$(find robot_ensamble_description)/meshes/Paleta_grid_1_1.stl" scale="0.001 0.001 0.001"/>
+      <mesh filename="$(arg mesh_prefix)Paleta_grid_1_1.stl" scale="0.001 0.001 0.001"/>
     </geometry>
   </collision>
@@ -253,5 +260,5 @@
     <origin xyz="-0.20388 -0.030969 -0.907" rpy="0 0 0"/>
     <geometry>
-      <mesh filename="file://$(find robot_ensamble_description)/meshes/Paleta_grid_2_1.stl" scale="0.001 0.001 0.001"/>
+      <mesh filename="$(arg mesh_prefix)Paleta_grid_2_1.stl" scale="0.001 0.001 0.001"/>
     </geometry>
     <material name="silver"/>
@@ -260,5 +267,5 @@
     <origin xyz="-0.20388 -0.030969 -0.907" rpy="0 0 0"/>
     <geometry>
-      <mesh filename="file://$(find robot_ensamble_description)/meshes/Paleta_grid_2_1.stl" scale="0.001 0.001 0.001"/>
+      <mesh filename="$(arg mesh_prefix)Paleta_grid_2_1.stl" scale="0.001 0.001 0.001"/>
     </geometry>
   </collision>
@@ -273,5 +280,5 @@
     <origin xyz="-0.214838 0.232986 -0.907" rpy="0 0 0"/>
     <geometry>
-      <mesh filename="file://$(find robot_ensamble_description)/meshes/Pala_DER_1.stl" scale="0.001 0.001 0.001"/>
+      <mesh filename="$(arg mesh_prefix)Pala_DER_1.stl" scale="0.001 0.001 0.001"/>
     </geometry>
     <material name="silver"/>
@@ -280,5 +287,5 @@
     <origin xyz="-0.214838 0.232986 -0.907" rpy="0 0 0"/>
     <geometry>
-      <mesh filename="file://$(find robot_ensamble_description)/meshes/Pala_DER_1.stl" scale="0.001 0.001 0.001"/>
+      <mesh filename="$(arg mesh_prefix)Pala_DER_1.stl" scale="0.001 0.001 0.001"/>
     </geometry>
   </collision>
@@ -293,5 +300,5 @@
     <origin xyz="-0.212742 -0.24501 -0.907" rpy="0 0 0"/>
     <geometry>
-      <mesh filename="file://$(find robot_ensamble_description)/meshes/Pala_IZQ_1.stl" scale="0.001 0.001 0.001"/>
+      <mesh filename="$(arg mesh_prefix)Pala_IZQ_1.stl" scale="0.001 0.001 0.001"/>
     </geometry>
     <material name="silver"/>
@@ -300,5 +307,5 @@
     <origin xyz="-0.212742 -0.24501 -0.907" rpy="0 0 0"/>
     <geometry>
-      <mesh filename="file://$(find robot_ensamble_description)/meshes/Pala_IZQ_1.stl" scale="0.001 0.001 0.001"/>
+      <mesh filename="$(arg mesh_prefix)Pala_IZQ_1.stl" scale="0.001 0.001 0.001"/>
     </geometry>
   </collision>
@@ -313,5 +320,5 @@
     <origin xyz="-0.211187 0.039037 -0.955" rpy="0 0 0"/>
     <geometry>
-      <mesh filename="file://$(find robot_ensamble_description)/meshes/Soporte_1_1.stl" scale="0.001 0.001 0.001"/>
+      <mesh filename="$(arg mesh_prefix)Soporte_1_1.stl" scale="0.001 0.001 0.001"/>
     </geometry>
     <material name="silver"/>
@@ -320,5 +327,5 @@
     <origin xyz="-0.211187 0.039037 -0.955" rpy="0 0 0"/>
     <geometry>
-      <mesh filename="file://$(find robot_ensamble_description)/meshes/Soporte_1_1.stl" scale="0.001 0.001 0.001"/>
+      <mesh filename="$(arg mesh_prefix)Soporte_1_1.stl" scale="0.001 0.001 0.001"/>
     </geometry>
   </collision>
@@ -333,5 +340,5 @@
     <origin xyz="-0.211187 0.038965 -0.859" rpy="0 0 0"/>
     <geometry>
-      <mesh filename="file://$(find robot_ensamble_description)/meshes/Soporte_2_1.stl" scale="0.001 0.001 0.001"/>
+      <mesh filename="$(arg mesh_prefix)Soporte_2_1.stl" scale="0.001 0.001 0.001"/>
     </geometry>
     <material name="silver"/>
@@ -340,10 +347,10 @@
     <origin xyz="-0.211187 0.038965 -0.859" rpy="0 0 0"/>
     <geometry>
-      <mesh filename="file://$(find robot_ensamble_description)/meshes/Soporte_2_1.stl" scale="0.001 0.001 0.001"/>
+      <mesh filename="$(arg mesh_prefix)Soporte_2_1.stl" scale="0.001 0.001 0.001"/>
     </geometry>
   </collision>
 </link>
 <joint name="x_link" type="prismatic">
-  <origin xyz="-0.02001 0.03 0.6215" rpy="0 0 0"/>
+  <origin xyz="-0.02001 0.031 0.6215" rpy="0 0 0"/>
   <parent link="base_link"/>
   <child link="x_link_1"/>
@@ -359,5 +366,5 @@
 </joint>
 <joint name="z_link" type="prismatic">
-  <origin xyz="0.005 0.0 0.0" rpy="0 0 0"/>
+  <origin xyz="0.005 0.0115 0.0" rpy="0 0 0"/>
   <parent link="y_link_1"/>
   <child link="z_link_1"/>
@@ -428,10 +435,10 @@
 </joint>
 <joint name="rig_9" type="fixed">
-  <origin xyz="0.000197 -0.045037 -0.033" rpy="0 0 0"/>
+  <origin xyz="0.000197 -0.32 -0.033" rpy="0 0 0"/>
   <parent link="cabezal_inferior_1"/>
   <child link="Soporte_1_1"/>
 </joint>
 <joint name="rig_10" type="fixed">
-  <origin xyz="0.000197 -0.044965 -0.129" rpy="0 0 0"/>
+  <origin xyz="0.000197 -0.32 -0.129" rpy="0 0 0"/>
   <parent link="cabezal_inferior_1"/>
   <child link="Soporte_2_1"/>
