Commit message: cambio color bandeja y se agrego urdf

File: src/bandeja_v3_description/urdf/bandeja_v3.xacro (robot description, xacro)
@@ -1,7 +1,12 @@
 <?xml version="1.0" ?>
 <robot name="bandeja_v3" xmlns:xacro="http://www.ros.org/wiki/xacro">
-<xacro:include filename="$(find bandeja_v3_description)/urdf/materials.xacro" />
-<xacro:include filename="$(find bandeja_v3_description)/urdf/bandeja_v3.trans" />
-<xacro:include filename="$(find bandeja_v3_description)/urdf/bandeja_v3.gazebo" />
+<xacro:arg name="include_ros_extensions" default="true"/>
+<xacro:arg name="mesh_directory" default="package://bandeja_v3_description/meshes"/>
+<xacro:property name="mesh_directory" value="$(arg mesh_directory)"/>
+<xacro:include filename="materials.xacro" />
+<xacro:if value="$(arg include_ros_extensions)">
+  <xacro:include filename="bandeja_v3.trans" />
+  <xacro:include filename="bandeja_v3.gazebo" />
+</xacro:if>
 <link name="base_link">
   <inertial>
@@ -13,5 +18,5 @@
     <origin xyz="0 0 0" rpy="0 0 0"/>
     <geometry>
-      <mesh filename="file://$(find bandeja_v3_description)/meshes/base_link.stl" scale="0.001 0.001 0.001"/>
+      <mesh filename="${mesh_directory}/base_link.stl" scale="0.001 0.001 0.001"/>
     </geometry>
     <material name="silver"/>
@@ -20,5 +25,5 @@
     <origin xyz="0 0 0" rpy="0 0 0"/>
     <geometry>
-      <mesh filename="file://$(find bandeja_v3_description)/meshes/base_link.stl" scale="0.001 0.001 0.001"/>
+      <mesh filename="${mesh_directory}/base_link.stl" scale="0.001 0.001 0.001"/>
     </geometry>
   </collision>

File: src/bandeja_v3_description/urdf/materials.xacro (robot description, xacro)
@@ -2,5 +2,5 @@
 <robot name="bandeja_v3" xmlns:xacro="http://www.ros.org/wiki/xacro" >
 <material name="silver">
-  <color rgba="0.700 0.700 0.700 1.000"/>
+  <color rgba="0.99 0.99 0.99 1.000"/>
 </material>
 </robot>
