Commit message: fix urdf robto_v2

File: src/robot_v2_description/urdf/robot_v2.urdf (robot description, URDF)
Before this commit: robot robot_v2, 18 links, 17 joints
Links:
- link Pala_DER_1: geometry collision mesh filename=package://robot_v2_description/meshes/Pala_DER_1.stl scale=0.001 0.001 0.001; visual mesh filename=package://robot_v2_description/meshes/Pala_DER_1.stl scale=0.001 0.001 0.001
- link Pala_IZQ_1: geometry collision mesh filename=package://robot_v2_description/meshes/Pala_IZQ_1.stl scale=0.001 0.001 0.001; visual mesh filename=package://robot_v2_description/meshes/Pala_IZQ_1.stl scale=0.001 0.001 0.001
- link Paleta_grid_1_1: geometry collision mesh filename=package://robot_v2_description/meshes/Paleta_grid_1_1.stl scale=0.001 0.001 0.001; visual mesh filename=package://robot_v2_description/meshes/Paleta_grid_1_1.stl scale=0.001 0.001 0.001
- link Paleta_grid_2_1: geometry collision mesh filename=package://robot_v2_description/meshes/Paleta_grid_2_1.stl scale=0.001 0.001 0.001; visual mesh filename=package://robot_v2_description/meshes/Paleta_grid_2_1.stl scale=0.001 0.001 0.001
- link Soporte_1_1: geometry collision mesh filename=package://robot_v2_description/meshes/Soporte_1_1.stl scale=0.001 0.001 0.001; visual mesh filename=package://robot_v2_description/meshes/Soporte_1_1.stl scale=0.001 0.001 0.001
- link Soporte_2_1: geometry collision mesh filename=package://robot_v2_description/meshes/Soporte_2_1.stl scale=0.001 0.001 0.001; visual mesh filename=package://robot_v2_description/meshes/Soporte_2_1.stl scale=0.001 0.001 0.001
- link acople_cabezal_1: geometry collision mesh filename=package://robot_v2_description/meshes/acople_cabezal_1.stl scale=0.001 0.001 0.001; visual mesh filename=package://robot_v2_description/meshes/acople_cabezal_1.stl scale=0.001 0.001 0.001
- link acople_palas_1: geometry collision mesh filename=package://robot_v2_description/meshes/acople_palas_1.stl scale=0.001 0.001 0.001; visual mesh filename=package://robot_v2_description/meshes/acople_palas_1.stl scale=0.001 0.001 0.001
- link base_link: geometry collision mesh filename=package://robot_v2_description/meshes/base_link.stl scale=0.001 0.001 0.001; visual mesh filename=package://robot_v2_description/meshes/base_link.stl scale=0.001 0.001 0.001
- link base_x_1: geometry collision mesh filename=package://robot_v2_description/meshes/base_x_1.stl scale=0.001 0.001 0.001; visual mesh filename=package://robot_v2_description/meshes/base_x_1.stl scale=0.001 0.001 0.001
- link cabezal_inferior_1: geometry collision mesh filename=package://robot_v2_description/meshes/cabezal_inferior_1.stl scale=0.001 0.001 0.001; visual mesh filename=package://robot_v2_description/meshes/cabezal_inferior_1.stl scale=0.001 0.001 0.001
- link complemento_cabezal_1: geometry collision mesh filename=package://robot_v2_description/meshes/complemento_cabezal_1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 scale=0.001 0.001 0.001; visual mesh filename=package://robot_v2_description/meshes/complemento_cabezal_1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 scale=0.001 0.001 0.001
- link horn_Servo_1: geometry collision mesh filename=package://robot_v2_description/meshes/horn_Servo_1.stl scale=0.001 0.001 0.001; visual mesh filename=package://robot_v2_description/meshes/horn_Servo_1.stl scale=0.001 0.001 0.001
- link robot_cabezal_1: geometry collision mesh filename=package://robot_v2_description/meshes/robot_cabezal_1.stl scale=0.001 0.001 0.001; visual mesh filename=package://robot_v2_description/meshes/robot_cabezal_1.stl scale=0.001 0.001 0.001
- link servo_mg996R_1: geometry collision mesh filename=package://robot_v2_description/meshes/servo_mg996R_1.stl scale=0.001 0.001 0.001; visual mesh filename=package://robot_v2_description/meshes/servo_mg996R_1.stl scale=0.001 0.001 0.001
- link x_link_1: geometry collision mesh filename=package://robot_v2_description/meshes/x_link_1.stl scale=0.001 0.001 0.001; visual mesh filename=package://robot_v2_description/meshes/x_link_1.stl scale=0.001 0.001 0.001
- link y_link_1: geometry collision mesh filename=package://robot_v2_description/meshes/y_link_1.stl scale=0.001 0.001 0.001; visual mesh filename=package://robot_v2_description/meshes/y_link_1.stl scale=0.001 0.001 0.001
- link z_link_1: geometry collision mesh filename=package://robot_v2_description/meshes/z_link_1.stl scale=0.001 0.001 0.001; visual mesh filename=package://robot_v2_description/meshes/z_link_1.stl scale=0.001 0.001 0.001

File: src/robot_v2_description/urdf/robot_v2.xacro (robot description, xacro)
@@ -1,7 +1,12 @@
 <?xml version="1.0" ?>
 <robot name="robot_v2" xmlns:xacro="http://www.ros.org/wiki/xacro">
-<xacro:include filename="$(find robot_v2_description)/urdf/materials.xacro" />
-<xacro:include filename="$(find robot_v2_description)/urdf/robot_v2.trans" />
-<xacro:include filename="$(find robot_v2_description)/urdf/robot_v2.gazebo" />
+<xacro:arg name="include_ros_extensions" default="true"/>
+<xacro:arg name="mesh_directory" default="package://robot_v2_description/meshes"/>
+<xacro:property name="mesh_directory" value="$(arg mesh_directory)"/>
+<xacro:include filename="materials.xacro" />
+<xacro:if value="$(arg include_ros_extensions)">
+  <xacro:include filename="robot_v2.trans" />
+  <xacro:include filename="robot_v2.gazebo" />
+</xacro:if>
 <link name="base_link">
   <inertial>
@@ -13,5 +18,5 @@
     <origin xyz="0 0 0" rpy="0 0 0"/>
     <geometry>
-      <mesh filename="file://$(find robot_v2_description)/meshes/base_link.stl" scale="0.001 0.001 0.001"/>
+      <mesh filename="${mesh_directory}/base_link.stl" scale="0.001 0.001 0.001"/>
     </geometry>
     <material name="gris_muy_oscuro"/>
@@ -20,5 +25,5 @@
     <origin xyz="0 0 0" rpy="0 0 0"/>
     <geometry>
-      <mesh filename="file://$(find robot_v2_description)/meshes/base_link.stl" scale="0.001 0.001 0.001"/>
+      <mesh filename="${mesh_directory}/base_link.stl" scale="0.001 0.001 0.001"/>
     </geometry>
   </collision>
@@ -33,5 +38,5 @@
     <origin xyz="-1.04 -0.0 -0.58" rpy="0 0 0"/>
     <geometry>
-      <mesh filename="file://$(find robot_v2_description)/meshes/base_x_1.stl" scale="0.001 0.001 0.001"/>
+      <mesh filename="${mesh_directory}/base_x_1.stl" scale="0.001 0.001 0.001"/>
     </geometry>
     <material name="plateado_metalico_brillante"/>
@@ -40,5 +45,5 @@
     <origin xyz="-1.04 -0.0 -0.58" rpy="0 0 0"/>
     <geometry>
-      <mesh filename="file://$(find robot_v2_description)/meshes/base_x_1.stl" scale="0.001 0.001 0.001"/>
+      <mesh filename="${mesh_directory}/base_x_1.stl" scale="0.001 0.001 0.001"/>
     </geometry>
   </collision>
@@ -53,5 +58,5 @@
     <origin xyz="-0.529995 -0.07 -0.6215" rpy="0 0 0"/>
     <geometry>
-      <mesh filename="file://$(find robot_v2_description)/meshes/x_link_1.stl" scale="0.001 0.001 0.001"/>
+      <mesh filename="${mesh_directory}/x_link_1.stl" scale="0.001 0.001 0.001"/>
     </geometry>
     <material name="plateado_metalico_brillante"/>
@@ -60,5 +65,5 @@
     <origin xyz="-0.529995 -0.07 -0.6215" rpy="0 0 0"/>
     <geometry>
-      <mesh filename="file://$(find robot_v2_description)/meshes/x_link_1.stl" scale="0.001 0.001 0.001"/>
+      <mesh filename="${mesh_directory}/x_link_1.stl" scale="0.001 0.001 0.001"/>
     </geometry>
   </collision>
@@ -73,5 +78,5 @@
     <origin xyz="-0.659995 -0.50041 -1.023" rpy="0 0 0"/>
     <geometry>
-      <mesh filename="file://$(find robot_v2_description)/meshes/y_link_1.stl" scale="0.001 0.001 0.001"/>
+      <mesh filename="${mesh_directory}/y_link_1.stl" scale="0.001 0.001 0.001"/>
     </geometry>
     <material name="negro_azabache_mate"/>
@@ -80,5 +85,5 @@
     <origin xyz="-0.659995 -0.50041 -1.023" rpy="0 0 0"/>
     <geometry>
-      <mesh filename="file://$(find robot_v2_description)/meshes/y_link_1.stl" scale="0.001 0.001 0.001"/>
+      <mesh filename="${mesh_directory}/y_link_1.stl" scale="0.001 0.001 0.001"/>
     </geometry>
   </collision>
@@ -93,5 +98,5 @@
     <origin xyz="-0.664995 -0.40041 -1.023" rpy="0 0 0"/>
     <geometry>
-      <mesh filename="file://$(find robot_v2_description)/meshes/z_link_1.stl" scale="0.001 0.001 0.001"/>
+      <mesh filename="${mesh_directory}/z_link_1.stl" scale="0.001 0.001 0.001"/>
     </geometry>
     <material name="plateado_metalico_brillante"/>
@@ -100,5 +105,5 @@
     <origin xyz="-0.664995 -0.40041 -1.023" rpy="0 0 0"/>
     <geometry>
-      <mesh filename="file://$(find robot_v2_description)/meshes/z_link_1.stl" scale="0.001 0.001 0.001"/>
+      <mesh filename="${mesh_directory}/z_link_1.stl" scale="0.001 0.001 0.001"/>
     </geometry>
   </collision>
@@ -113,5 +118,5 @@
     <origin xyz="-0.704995 -0.43891 -1.023" rpy="0 0 0"/>
     <geometry>
-      <mesh filename="file://$(find robot_v2_description)/meshes/complemento_cabezal_1.stl" scale="0.001 0.001 0.001"/>
+      <mesh filename="${mesh_directory}/complemento_cabezal_1.stl" scale="0.001 0.001 0.001"/>
     </geometry>
     <material name="verde"/>
@@ -120,5 +125,5 @@
     <origin xyz="-0.704995 -0.43891 -1.023" rpy="0 0 0"/>
     <geometry>
-      <mesh filename="file://$(find robot_v2_description)/meshes/complemento_cabezal_1.stl" scale="0.001 0.001 0.001"/>
+      <mesh filename="${mesh_directory}/complemento_cabezal_1.stl" scale="0.001 0.001 0.001"/>
     </geometry>
   </collision>
@@ -133,5 +138,5 @@
     <origin xyz="-0.710995 -0.43891 -1.023" rpy="0 0 0"/>
     <geometry>
-      <mesh filename="file://$(find robot_v2_description)/meshes/robot_cabezal_1.stl" scale="0.001 0.001 0.001"/>
+      <mesh filename="${mesh_directory}/robot_cabezal_1.stl" scale="0.001 0.001 0.001"/>
     </geometry>
     <material name="negro_azabache_mate"/>
@@ -140,5 +145,5 @@
     <origin xyz="-0.710995 -0.43891 -1.023" rpy="0 0 0"/>
     <geometry>
-      <mesh filename="file://$(find robot_v2_description)/meshes/robot_cabezal_1.stl" scale="0.001 0.001 0.001"/>
+      <mesh filename="${mesh_directory}/robot_cabezal_1.stl" scale="0.001 0.001 0.001"/>
     </geometry>
   </collision>
@@ -153,5 +158,5 @@
     <origin xyz="-0.760995 -0.43891 -1.0455" rpy="0 0 0"/>
     <geometry>
-      <mesh filename="file://$(find robot_v2_description)/meshes/acople_cabezal_1.stl" scale="0.001 0.001 0.001"/>
+      <mesh filename="${mesh_directory}/acople_cabezal_1.stl" scale="0.001 0.001 0.001"/>
     </geometry>
     <material name="negro_azabache_mate"/>
@@ -160,5 +165,5 @@
     <origin xyz="-0.760995 -0.43891 -1.0455" rpy="0 0 0"/>
     <geometry>
-      <mesh filename="file://$(find robot_v2_description)/meshes/acople_cabezal_1.stl" scale="0.001 0.001 0.001"/>
+      <mesh filename="${mesh_directory}/acople_cabezal_1.stl" scale="0.001 0.001 0.001"/>
     </geometry>
   </collision>
@@ -173,5 +178,5 @@
     <origin xyz="-0.760995 -0.43891 -0.996" rpy="0 0 0"/>
     <geometry>
-      <mesh filename="file://$(find robot_v2_description)/meshes/cabezal_inferior_1.stl" scale="0.001 0.001 0.001"/>
+      <mesh filename="${mesh_directory}/cabezal_inferior_1.stl" scale="0.001 0.001 0.001"/>
     </geometry>
     <material name="azul_violaceo"/>
@@ -180,5 +185,5 @@
     <origin xyz="-0.760995 -0.43891 -0.996" rpy="0 0 0"/>
     <geometry>
-      <mesh filename="file://$(find robot_v2_description)/meshes/cabezal_inferior_1.stl" scale="0.001 0.001 0.001"/>
+      <mesh filename="${mesh_directory}/cabezal_inferior_1.stl" scale="0.001 0.001 0.001"/>
     </geometry>
   </collision>
@@ -193,5 +198,5 @@
     <origin xyz="-0.740517 -0.43382 -0.8805" rpy="0 0 0"/>
     <geometry>
-      <mesh filename="file://$(find robot_v2_description)/meshes/servo_mg996R_1.stl" scale="0.001 0.001 0.001"/>
+      <mesh filename="${mesh_directory}/servo_mg996R_1.stl" scale="0.001 0.001 0.001"/>
     </geometry>
     <material name="negro_azabache_mate"/>
@@ -200,5 +205,5 @@
     <origin xyz="-0.740517 -0.43382 -0.8805" rpy="0 0 0"/>
     <geometry>
-      <mesh filename="file://$(find robot_v2_description)/meshes/servo_mg996R_1.stl" scale="0.001 0.001 0.001"/>
+      <mesh filename="${mesh_directory}/servo_mg996R_1.stl" scale="0.001 0.001 0.001"/>
     </geometry>
   </collision>
@@ -208,10 +213,11 @@
     <origin xyz="0.003187489121206477 1.4413294837922752e-05 0.0" rpy="0 0 0"/>
     <mass value="0.005099610361289279"/>
-    <inertia ixx="0.0" iyy="0.0" izz="0.0" ixy="0.0" iyz="0.0" ixz="0.0"/>
+    <!-- Estimacion por volumen STL y densidad uniforme; masa y origen CAD conservados. -->
+    <inertia ixx="2.4043669365e-07" iyy="1.2530990893e-07" izz="1.25307578e-07" ixy="5.0476408546e-10" iyz="2.4855236723e-15" ixz="-8.5505096321e-16"/>
   </inertial>
   <visual>
     <origin xyz="-0.752495 -0.438872 -0.915" rpy="0 0 0"/>
     <geometry>
-      <mesh filename="file://$(find robot_v2_description)/meshes/horn_Servo_1.stl" scale="0.001 0.001 0.001"/>
+      <mesh filename="${mesh_directory}/horn_Servo_1.stl" scale="0.001 0.001 0.001"/>
     </geometry>
     <material name="negro_azabache_mate"/>
@@ -220,5 +226,5 @@
     <origin xyz="-0.752495 -0.438872 -0.915" rpy="0 0 0"/>
     <geometry>
-      <mesh filename="file://$(find robot_v2_description)/meshes/horn_Servo_1.stl" scale="0.001 0.001 0.001"/>
+      <mesh filename="${mesh_directory}/horn_Servo_1.stl" scale="0.001 0.001 0.001"/>
     </geometry>
   </collision>
@@ -233,5 +239,5 @@
     <origin xyz="-0.756995 -0.438892 -0.915" rpy="0 0 0"/>
     <geometry>
-      <mesh filename="file://$(find robot_v2_description)/meshes/acople_palas_1.stl" scale="0.001 0.001 0.001"/>
+      <mesh filename="${mesh_directory}/acople_palas_1.stl" scale="0.001 0.001 0.001"/>
     </geometry>
     <material name="negro_azabache_mate"/>
@@ -240,5 +246,5 @@
     <origin xyz="-0.756995 -0.438892 -0.915" rpy="0 0 0"/>
     <geometry>
-      <mesh filename="file://$(find robot_v2_description)/meshes/acople_palas_1.stl" scale="0.001 0.001 0.001"/>
+      <mesh filename="${mesh_directory}/acople_palas_1.stl" scale="0.001 0.001 0.001"/>
     </geometry>
   </collision>
@@ -253,5 +259,5 @@
     <origin xyz="-0.754105 -0.413879 -0.915" rpy="0 0 0"/>
     <geometry>
-      <mesh filename="file://$(find robot_v2_description)/meshes/Paleta_grid_1_1.stl" scale="0.001 0.001 0.001"/>
+      <mesh filename="${mesh_directory}/Paleta_grid_1_1.stl" scale="0.001 0.001 0.001"/>
     </geometry>
     <material name="negro_azabache_mate"/>
@@ -260,5 +266,5 @@
     <origin xyz="-0.754105 -0.413879 -0.915" rpy="0 0 0"/>
     <geometry>
-      <mesh filename="file://$(find robot_v2_description)/meshes/Paleta_grid_1_1.stl" scale="0.001 0.001 0.001"/>
+      <mesh filename="${mesh_directory}/Paleta_grid_1_1.stl" scale="0.001 0.001 0.001"/>
     </geometry>
   </collision>
@@ -273,5 +279,5 @@
     <origin xyz="-0.753885 -0.463879 -0.915" rpy="0 0 0"/>
     <geometry>
-      <mesh filename="file://$(find robot_v2_description)/meshes/Paleta_grid_2_1.stl" scale="0.001 0.001 0.001"/>
+      <mesh filename="${mesh_directory}/Paleta_grid_2_1.stl" scale="0.001 0.001 0.001"/>
     </geometry>
     <material name="negro_azabache_mate"/>
@@ -280,5 +286,5 @@
     <origin xyz="-0.753885 -0.463879 -0.915" rpy="0 0 0"/>
     <geometry>
-      <mesh filename="file://$(find robot_v2_description)/meshes/Paleta_grid_2_1.stl" scale="0.001 0.001 0.001"/>
+      <mesh filename="${mesh_directory}/Paleta_grid_2_1.stl" scale="0.001 0.001 0.001"/>
     </geometry>
   </collision>
@@ -293,5 +299,5 @@
     <origin xyz="-0.764843 -0.199924 -0.915" rpy="0 0 0"/>
     <geometry>
-      <mesh filename="file://$(find robot_v2_description)/meshes/Pala_DER_1.stl" scale="0.001 0.001 0.001"/>
+      <mesh filename="${mesh_directory}/Pala_DER_1.stl" scale="0.001 0.001 0.001"/>
     </geometry>
     <material name="cafe_oscuro"/>
@@ -300,5 +306,5 @@
     <origin xyz="-0.764843 -0.199924 -0.915" rpy="0 0 0"/>
     <geometry>
-      <mesh filename="file://$(find robot_v2_description)/meshes/Pala_DER_1.stl" scale="0.001 0.001 0.001"/>
+      <mesh filename="${mesh_directory}/Pala_DER_1.stl" scale="0.001 0.001 0.001"/>
     </geometry>
   </collision>
@@ -313,5 +319,5 @@
     <origin xyz="-0.762747 -0.67792 -0.915" rpy="0 0 0"/>
     <geometry>
-      <mesh filename="file://$(find robot_v2_description)/meshes/Pala_IZQ_1.stl" scale="0.001 0.001 0.001"/>
+      <mesh filename="${mesh_directory}/Pala_IZQ_1.stl" scale="0.001 0.001 0.001"/>
     </geometry>
     <material name="cafe_oscuro"/>
@@ -320,5 +326,5 @@
     <origin xyz="-0.762747 -0.67792 -0.915" rpy="0 0 0"/>
     <geometry>
-      <mesh filename="file://$(find robot_v2_description)/meshes/Pala_IZQ_1.stl" scale="0.001 0.001 0.001"/>
+      <mesh filename="${mesh_directory}/Pala_IZQ_1.stl" scale="0.001 0.001 0.001"/>
     </geometry>
   </collision>
@@ -328,10 +334,11 @@
     <origin xyz="-0.001402560565108013 0.31999688228192996 -1.1102230246251565e-16" rpy="0 0 0"/>
     <mass value="0.02663442251713428"/>
-    <inertia ixx="0.000909" iyy="0.0" izz="0.000909" ixy="4e-06" iyz="0.0" ixz="0.0"/>
+    <!-- Estimacion por volumen STL y densidad uniforme; masa y origen CAD conservados. -->
+    <inertia ixx="0.00092037155027" iyy="3.1003731189e-07" izz="0.00092038912539" ixy="4.0340583526e-06" iyz="-3.1255448549e-12" ixz="2.5007250268e-14"/>
   </inertial>
   <visual>
     <origin xyz="-0.761192 -0.393873 -0.963" rpy="0 0 0"/>
     <geometry>
-      <mesh filename="file://$(find robot_v2_description)/meshes/Soporte_1_1.stl" scale="0.001 0.001 0.001"/>
+      <mesh filename="${mesh_directory}/Soporte_1_1.stl" scale="0.001 0.001 0.001"/>
     </geometry>
     <material name="silver"/>
@@ -340,5 +347,5 @@
     <origin xyz="-0.761192 -0.393873 -0.963" rpy="0 0 0"/>
     <geometry>
-      <mesh filename="file://$(find robot_v2_description)/meshes/Soporte_1_1.stl" scale="0.001 0.001 0.001"/>
+      <mesh filename="${mesh_directory}/Soporte_1_1.stl" scale="0.001 0.001 0.001"/>
     </geometry>
   </collision>
@@ -348,10 +355,11 @@
     <origin xyz="-0.0014028765290923229 0.3199969462788138 -2.220446049250313e-16" rpy="0 0 0"/>
     <mass value="0.02663442251713428"/>
-    <inertia ixx="0.000909" iyy="0.0" izz="0.000909" ixy="4e-06" iyz="0.0" ixz="0.0"/>
+    <!-- Estimacion por volumen STL y densidad uniforme; masa y origen CAD conservados. -->
+    <inertia ixx="0.00092037233368" iyy="3.1003779368e-07" izz="0.0009203899093" ixy="4.0341053871e-06" iyz="1.8476833119e-13" ixz="-1.0493772854e-14"/>
   </inertial>
   <visual>
     <origin xyz="-0.761192 -0.393945 -0.867" rpy="0 0 0"/>
     <geometry>
-      <mesh filename="file://$(find robot_v2_description)/meshes/Soporte_2_1.stl" scale="0.001 0.001 0.001"/>
+      <mesh filename="${mesh_directory}/Soporte_2_1.stl" scale="0.001 0.001 0.001"/>
     </geometry>
     <material name="silver"/>
@@ -360,5 +368,5 @@
     <origin xyz="-0.761192 -0.393945 -0.867" rpy="0 0 0"/>
     <geometry>
-      <mesh filename="file://$(find robot_v2_description)/meshes/Soporte_2_1.stl" scale="0.001 0.001 0.001"/>
+      <mesh filename="${mesh_directory}/Soporte_2_1.stl" scale="0.001 0.001 0.001"/>
     </geometry>
   </collision>
